File: Stepper_Control.kicad_sch (KiCad schematic)
At the start: 1 part, among them J701 2350514-8

Commit message: update schematique
Parts:
- renumbered J701 to J15
Changed lines of the file:
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@@
 		(dnp no)
 		(fields_autoplaced yes)
-		(property "Reference" "J701"
+		(property "Reference" "J15"
 			(at 167.64 78.7399 0)
 			(effects
@@
 			(project "SACE-HW"
 				(path "/4c1e5ca8-aa0f-4a8e-bffe-6765adb2e3e8/114a8538-54a0-4526-bfdc-fea8737f7836"
-					(reference "J701")
+					(reference "J15")
 					(unit 1)
 				)
