File: 5V_OUTPUT.kicad_sch (KiCad schematic)
At the start: 4 parts, among them J701 2350514-8, U701 74LVC4245APW_118

Commit message: update schematic
Parts:
- renumbered C701 to C38, C702 to C39, J701 to J17, U701 to U16
Changed lines of the file:
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@@
 	)
 	(hierarchical_label "OUT7"
-		(shape output)
+		(shape input)
 		(at 104.14 102.87 180)
 		(fields_autoplaced yes)
@@
 	)
 	(hierarchical_label "OUT1"
-		(shape output)
+		(shape input)
 		(at 104.14 87.63 180)
 		(fields_autoplaced yes)
@@
 	)
 	(hierarchical_label "OUT2"
-		(shape output)
+		(shape input)
 		(at 104.14 90.17 180)
 		(fields_autoplaced yes)
@@
 	)
 	(hierarchical_label "OUT4"
-		(shape output)
+		(shape input)
 		(at 104.14 95.25 180)
 		(fields_autoplaced yes)
@@
 	)
 	(hierarchical_label "OUT6"
-		(shape output)
+		(shape input)
 		(at 104.14 100.33 180)
 		(fields_autoplaced yes)
@@
 	)
 	(hierarchical_label "OUT3"
-		(shape output)
+		(shape input)
 		(at 104.14 92.71 180)
 		(fields_autoplaced yes)
@@
 	)
 	(hierarchical_label "OUT5"
-		(shape output)
+		(shape input)
 		(at 104.14 97.79 180)
 		(fields_autoplaced yes)
@@
 	)
 	(hierarchical_label "OUT0"
-		(shape output)
+		(shape input)
 		(at 104.14 85.09 180)
 		(fields_autoplaced yes)
@@
 		(dnp no)
 		(fields_autoplaced yes)
-		(property "Reference" "#PWR0704"
+		(property "Reference" "#PWR0131"
 			(at 171.45 71.12 0)
 			(effects
@@
 			(project "SACE-HW"
 				(path "/4c1e5ca8-aa0f-4a8e-bffe-6765adb2e3e8/114a8538-54a0-4526-bfdc-fea8737f7836"
-					(reference "#PWR0704")
+					(reference "#PWR0131")
 					(unit 1)
 				)
@@
 		(on_board yes)
 		(dnp no)
-		(property "Reference" "C701"
+		(property "Reference" "C38"
 			(at 162.052 69.088 90)
 			(effects
@@
 			(project "SACE-HW"
 				(path "/4c1e5ca8-aa0f-4a8e-bffe-6765adb2e3e8/114a8538-54a0-4526-bfdc-fea8737f7836"
-					(reference "C701")
+					(reference "C38")
 					(unit 1)
 				)
@@
 		(on_board yes)
 		(dnp no)
-		(property "Reference" "#PWR0706"
+		(property "Reference" "#PWR0127"
 			(at 138.43 84.328 0)
 			(effects
@@
 			(project "SACE-HW"
 				(path "/4c1e5ca8-aa0f-4a8e-bffe-6765adb2e3e8/114a8538-54a0-4526-bfdc-fea8737f7836"
-					(reference "#PWR0706")
+					(reference "#PWR0127")
 					(unit 1)
 				)
@@
 		(on_board yes)
 		(dnp no)
-		(property "Reference" "#PWR0705"
+		(property "Reference" "#PWR0130"
 			(at 166.37 83.058 0)
 			(effects
@@
 			(project "SACE-HW"
 				(path "/4c1e5ca8-aa0f-4a8e-bffe-6765adb2e3e8/114a8538-54a0-4526-bfdc-fea8737f7836"
-					(reference "#PWR0705")
+					(reference "#PWR0130")
 					(unit 1)
 				)
@@
 		(on_board yes)
 		(dnp no)
-		(property "Reference" "#PWR0707"
+		(property "Reference" "#PWR0126"
 			(at 134.62 121.158 0)
 			(effects
@@
 			(project "SACE-HW"
 				(path "/4c1e5ca8-aa0f-4a8e-bffe-6765adb2e3e8/114a8538-54a0-4526-bfdc-fea8737f7836"
-					(reference "#PWR0707")
+					(reference "#PWR0126")
 					(unit 1)
 				)
@@
 		(on_board yes)
 		(dnp no)
-		(property "Reference" "U701"
+		(property "Reference" "U16"
 			(at 120.65 59.69 0)
 			(effects
@@
 			(project "SACE-HW"
 				(path "/4c1e5ca8-aa0f-4a8e-bffe-6765adb2e3e8/114a8538-54a0-4526-bfdc-fea8737f7836"
-					(reference "U701")
+					(reference "U16")
 					(unit 1)
 				)
@@
 		(on_board yes)
 		(dnp no)
-		(property "Reference" "C702"
+		(property "Reference" "C39"
 			(at 172.72 68.834 90)
 			(effects
@@
 			(project "SACE-HW"
 				(path "/4c1e5ca8-aa0f-4a8e-bffe-6765adb2e3e8/114a8538-54a0-4526-bfdc-fea8737f7836"
-					(reference "C702")
+					(reference "C39")
 					(unit 1)
 				)
@@
 		(dnp no)
 		(fields_autoplaced yes)
-		(property "Reference" "#PWR0703"
+		(property "Reference" "#PWR0129"
 			(at 161.29 71.12 0)
 			(effects
@@
 			(project "SACE-HW"
 				(path "/4c1e5ca8-aa0f-4a8e-bffe-6765adb2e3e8/114a8538-54a0-4526-bfdc-fea8737f7836"
-					(reference "#PWR0703")
+					(reference "#PWR0129")
 					(unit 1)
 				)
@@
 		(dnp no)
 		(fields_autoplaced yes)
-		(property "Reference" "#PWR0702"
+		(property "Reference" "#PWR0128"
 			(at 142.24 71.12 0)
 			(effects
@@
 			(project "SACE-HW"
 				(path "/4c1e5ca8-aa0f-4a8e-bffe-6765adb2e3e8/114a8538-54a0-4526-bfdc-fea8737f7836"
-					(reference "#PWR0702")
+					(reference "#PWR0128")
 					(unit 1)
 				)
@@
 		(dnp no)
 		(fields_autoplaced yes)
-		(property "Reference" "#PWR0701"
+		(property "Reference" "#PWR0125"
 			(at 134.62 71.12 0)
 			(effects
@@
 			(project "SACE-HW"
 				(path "/4c1e5ca8-aa0f-4a8e-bffe-6765adb2e3e8/114a8538-54a0-4526-bfdc-fea8737f7836"
-					(reference "#PWR0701")
+					(reference "#PWR0125")
 					(unit 1)
 				)
@@
 		(dnp no)
 		(fields_autoplaced yes)
-		(property "Reference" "J701"
+		(property "Reference" "J17"
 			(at 153.67 93.9799 0)
 			(effects
@@
 			(project "SACE-HW"
 				(path "/4c1e5ca8-aa0f-4a8e-bffe-6765adb2e3e8/114a8538-54a0-4526-bfdc-fea8737f7836"
-					(reference "J701")
+					(reference "J17")
 					(unit 1)
 				)

Commit message: finalisation de la schématique
Parts:
- renumbered C38 to C701, C39 to C702, J17 to J701, U16 to U701
Changed lines of the file:
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@@
 		(dnp no)
 		(fields_autoplaced yes)
-		(property "Reference" "#PWR0131"
+		(property "Reference" "#PWR0704"
 			(at 171.45 71.12 0)
 			(effects
@@
 			(project "SACE-HW"
 				(path "/4c1e5ca8-aa0f-4a8e-bffe-6765adb2e3e8/114a8538-54a0-4526-bfdc-fea8737f7836"
-					(reference "#PWR0131")
+					(reference "#PWR0704")
 					(unit 1)
 				)
@@
 		(on_board yes)
 		(dnp no)
-		(property "Reference" "C38"
+		(property "Reference" "C701"
 			(at 162.052 69.088 90)
 			(effects
@@
 			(project "SACE-HW"
 				(path "/4c1e5ca8-aa0f-4a8e-bffe-6765adb2e3e8/114a8538-54a0-4526-bfdc-fea8737f7836"
-					(reference "C38")
+					(reference "C701")
 					(unit 1)
 				)
@@
 		(on_board yes)
 		(dnp no)
-		(property "Reference" "#PWR0127"
+		(property "Reference" "#PWR0706"
 			(at 138.43 84.328 0)
 			(effects
@@
 			(project "SACE-HW"
 				(path "/4c1e5ca8-aa0f-4a8e-bffe-6765adb2e3e8/114a8538-54a0-4526-bfdc-fea8737f7836"
-					(reference "#PWR0127")
+					(reference "#PWR0706")
 					(unit 1)
 				)
@@
 		(on_board yes)
 		(dnp no)
-		(property "Reference" "#PWR0130"
+		(property "Reference" "#PWR0705"
 			(at 166.37 83.058 0)
 			(effects
@@
 			(project "SACE-HW"
 				(path "/4c1e5ca8-aa0f-4a8e-bffe-6765adb2e3e8/114a8538-54a0-4526-bfdc-fea8737f7836"
-					(reference "#PWR0130")
+					(reference "#PWR0705")
 					(unit 1)
 				)
@@
 		(on_board yes)
 		(dnp no)
-		(property "Reference" "#PWR0126"
+		(property "Reference" "#PWR0707"
 			(at 134.62 121.158 0)
 			(effects
@@
 			(project "SACE-HW"
 				(path "/4c1e5ca8-aa0f-4a8e-bffe-6765adb2e3e8/114a8538-54a0-4526-bfdc-fea8737f7836"
-					(reference "#PWR0126")
+					(reference "#PWR0707")
 					(unit 1)
 				)
@@
 		(on_board yes)
 		(dnp no)
-		(property "Reference" "U16"
+		(property "Reference" "U701"
 			(at 120.65 59.69 0)
 			(effects
@@
 			(project "SACE-HW"
 				(path "/4c1e5ca8-aa0f-4a8e-bffe-6765adb2e3e8/114a8538-54a0-4526-bfdc-fea8737f7836"
-					(reference "U16")
+					(reference "U701")
 					(unit 1)
 				)
@@
 		(on_board yes)
 		(dnp no)
-		(property "Reference" "C39"
+		(property "Reference" "C702"
 			(at 172.72 68.834 90)
 			(effects
@@
 			(project "SACE-HW"
 				(path "/4c1e5ca8-aa0f-4a8e-bffe-6765adb2e3e8/114a8538-54a0-4526-bfdc-fea8737f7836"
-					(reference "C39")
+					(reference "C702")
 					(unit 1)
 				)
@@
 		(dnp no)
 		(fields_autoplaced yes)
-		(property "Reference" "#PWR0129"
+		(property "Reference" "#PWR0703"
 			(at 161.29 71.12 0)
 			(effects
@@
 			(project "SACE-HW"
 				(path "/4c1e5ca8-aa0f-4a8e-bffe-6765adb2e3e8/114a8538-54a0-4526-bfdc-fea8737f7836"
-					(reference "#PWR0129")
+					(reference "#PWR0703")
 					(unit 1)
 				)
@@
 		(dnp no)
 		(fields_autoplaced yes)
-		(property "Reference" "#PWR0128"
+		(property "Reference" "#PWR0702"
 			(at 142.24 71.12 0)
 			(effects
@@
 			(project "SACE-HW"
 				(path "/4c1e5ca8-aa0f-4a8e-bffe-6765adb2e3e8/114a8538-54a0-4526-bfdc-fea8737f7836"
-					(reference "#PWR0128")
+					(reference "#PWR0702")
 					(unit 1)
 				)
@@
 		(dnp no)
 		(fields_autoplaced yes)
-		(property "Reference" "#PWR0125"
+		(property "Reference" "#PWR0701"
 			(at 134.62 71.12 0)
 			(effects
@@
 			(project "SACE-HW"
 				(path "/4c1e5ca8-aa0f-4a8e-bffe-6765adb2e3e8/114a8538-54a0-4526-bfdc-fea8737f7836"
-					(reference "#PWR0125")
+					(reference "#PWR0701")
 					(unit 1)
 				)
@@
 		(dnp no)
 		(fields_autoplaced yes)
-		(property "Reference" "J17"
+		(property "Reference" "J701"
 			(at 153.67 93.9799 0)
 			(effects
@@
 			(project "SACE-HW"
 				(path "/4c1e5ca8-aa0f-4a8e-bffe-6765adb2e3e8/114a8538-54a0-4526-bfdc-fea8737f7836"
-					(reference "J17")
-					(unit 1)
-				)
+					(reference "J701")
+					(unit 1)
+				)

Commit message: update
Parts:
- renumbered C701 to C601, C702 to C602, J701 to J601, U701 to U601
Changed lines of the file:
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@@
 		(dnp no)
 		(fields_autoplaced yes)
-		(property "Reference" "#PWR0704"
+		(property "Reference" "#PWR0604"
 			(at 171.45 71.12 0)
 			(effects
@@
 			(project "SACE-HW"
 				(path "/4c1e5ca8-aa0f-4a8e-bffe-6765adb2e3e8/114a8538-54a0-4526-bfdc-fea8737f7836"
-					(reference "#PWR0704")
+					(reference "#PWR0604")
 					(unit 1)
 				)
@@
 		(on_board yes)
 		(dnp no)
-		(property "Reference" "C701"
+		(property "Reference" "C601"
 			(at 162.052 69.088 90)
 			(effects
@@
 			(project "SACE-HW"
 				(path "/4c1e5ca8-aa0f-4a8e-bffe-6765adb2e3e8/114a8538-54a0-4526-bfdc-fea8737f7836"
-					(reference "C701")
+					(reference "C601")
 					(unit 1)
 				)
@@
 		(on_board yes)
 		(dnp no)
-		(property "Reference" "#PWR0706"
+		(property "Reference" "#PWR0606"
 			(at 138.43 84.328 0)
 			(effects
@@
 			(project "SACE-HW"
 				(path "/4c1e5ca8-aa0f-4a8e-bffe-6765adb2e3e8/114a8538-54a0-4526-bfdc-fea8737f7836"
-					(reference "#PWR0706")
+					(reference "#PWR0606")
 					(unit 1)
 				)
@@
 		(on_board yes)
 		(dnp no)
-		(property "Reference" "#PWR0705"
+		(property "Reference" "#PWR0605"
 			(at 166.37 83.058 0)
 			(effects
@@
 			(project "SACE-HW"
 				(path "/4c1e5ca8-aa0f-4a8e-bffe-6765adb2e3e8/114a8538-54a0-4526-bfdc-fea8737f7836"
-					(reference "#PWR0705")
+					(reference "#PWR0605")
 					(unit 1)
 				)
@@
 		(on_board yes)
 		(dnp no)
-		(property "Reference" "#PWR0707"
+		(property "Reference" "#PWR0607"
 			(at 134.62 121.158 0)
 			(effects
@@
 			(project "SACE-HW"
 				(path "/4c1e5ca8-aa0f-4a8e-bffe-6765adb2e3e8/114a8538-54a0-4526-bfdc-fea8737f7836"
-					(reference "#PWR0707")
+					(reference "#PWR0607")
 					(unit 1)
 				)
@@
 		(on_board yes)
 		(dnp no)
-		(property "Reference" "U701"
+		(property "Reference" "U601"
 			(at 120.65 59.69 0)
 			(effects
@@
 			(project "SACE-HW"
 				(path "/4c1e5ca8-aa0f-4a8e-bffe-6765adb2e3e8/114a8538-54a0-4526-bfdc-fea8737f7836"
-					(reference "U701")
+					(reference "U601")
 					(unit 1)
 				)
@@
 		(on_board yes)
 		(dnp no)
-		(property "Reference" "C702"
+		(property "Reference" "C602"
 			(at 172.72 68.834 90)
 			(effects
@@
 			(project "SACE-HW"
 				(path "/4c1e5ca8-aa0f-4a8e-bffe-6765adb2e3e8/114a8538-54a0-4526-bfdc-fea8737f7836"
-					(reference "C702")
+					(reference "C602")
 					(unit 1)
 				)
@@
 		(dnp no)
 		(fields_autoplaced yes)
-		(property "Reference" "#PWR0703"
+		(property "Reference" "#PWR0603"
 			(at 161.29 71.12 0)
 			(effects
@@
 			(project "SACE-HW"
 				(path "/4c1e5ca8-aa0f-4a8e-bffe-6765adb2e3e8/114a8538-54a0-4526-bfdc-fea8737f7836"
-					(reference "#PWR0703")
+					(reference "#PWR0603")
 					(unit 1)
 				)
@@
 		(dnp no)
 		(fields_autoplaced yes)
-		(property "Reference" "#PWR0702"
+		(property "Reference" "#PWR0602"
 			(at 142.24 71.12 0)
 			(effects
@@
 			(project "SACE-HW"
 				(path "/4c1e5ca8-aa0f-4a8e-bffe-6765adb2e3e8/114a8538-54a0-4526-bfdc-fea8737f7836"
-					(reference "#PWR0702")
+					(reference "#PWR0602")
 					(unit 1)
 				)
@@
 		(dnp no)
 		(fields_autoplaced yes)
-		(property "Reference" "#PWR0701"
+		(property "Reference" "#PWR0601"
 			(at 134.62 71.12 0)
 			(effects
@@
 			(project "SACE-HW"
 				(path "/4c1e5ca8-aa0f-4a8e-bffe-6765adb2e3e8/114a8538-54a0-4526-bfdc-fea8737f7836"
-					(reference "#PWR0701")
+					(reference "#PWR0601")
 					(unit 1)
 				)
@@
 		(dnp no)
 		(fields_autoplaced yes)
-		(property "Reference" "J701"
+		(property "Reference" "J601"
 			(at 153.67 93.9799 0)
 			(effects
@@
 			(project "SACE-HW"
 				(path "/4c1e5ca8-aa0f-4a8e-bffe-6765adb2e3e8/114a8538-54a0-4526-bfdc-fea8737f7836"
-					(reference "J701")
-					(unit 1)
-				)
+					(reference "J601")
+					(unit 1)
+				)
