File: HV.kicad_sch (KiCad schematic)
At the start: 29 parts, among them J401 1935161, J402 1935161, J403 RF1-01K-D-00-50-BK-HDW, J404 RF1-01K-D-00-50-BK-HDW, Q401 MCB90N12A-TP, U401 LTV-816S, U402 ADC124S021CIMM, U403 TMCS1101A3UQDT, U404 ISO7341CQDWQ1, U405 MCP6L04T-E/SL

Commit message: clean up
Other:
- moved on the sheet: U404
Changed lines of the file:
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@@
 	)
 	(no_connect
-		(at 190.5 119.38)
+		(at 217.17 119.38)
 	)
 	(no_connect
@@
 	)
 	(no_connect
-		(at 215.9 119.38)
+		(at 191.77 119.38)
 	)
 	(no_connect
@@
 	(wire
 		(pts
-			(xy 215.9 88.9) (xy 218.44 88.9)
+			(xy 191.77 88.9) (xy 189.23 88.9)
 		)
 		(stroke
@@
 	(wire
 		(pts
-			(xy 215.9 93.98) (xy 228.6 93.98)
+			(xy 191.77 93.98) (xy 179.07 93.98)
 		)
 		(stroke
@@
 	(wire
 		(pts
-			(xy 215.9 109.22) (xy 223.52 109.22)
+			(xy 191.77 109.22) (xy 184.15 109.22)
 		)
 		(stroke
@@
 	(wire
 		(pts
-			(xy 215.9 104.14) (xy 223.52 104.14)
+			(xy 191.77 104.14) (xy 184.15 104.14)
 		)
 		(stroke
@@
 	(wire
 		(pts
-			(xy 190.5 93.98) (xy 179.07 93.98)
+			(xy 217.17 93.98) (xy 228.6 93.98)
 		)
 		(stroke
@@
 	(wire
 		(pts
-			(xy 189.23 88.9) (xy 190.5 88.9)
+			(xy 218.44 88.9) (xy 217.17 88.9)
 		)
 		(stroke
@@
 	(wire
 		(pts
-			(xy 215.9 99.06) (xy 223.52 99.06)
+			(xy 191.77 99.06) (xy 184.15 99.06)
 		)
 		(stroke
@@
 	(wire
 		(pts
-			(xy 215.9 114.3) (xy 223.52 114.3)
+			(xy 191.77 114.3) (xy 184.15 114.3)
 		)
 		(stroke
@@
 	)
 	(label "CS_A"
-		(at 223.52 104.14 180)
+		(at 184.15 104.14 0)
 		(fields_autoplaced yes)
 		(effects
@@
 				(size 1.27 1.27)
 			)
-			(justify right bottom)
+			(justify left bottom)
 		)
 	)
@@
 	)
 	(label "MISO_A"
-		(at 223.52 114.3 180)
+		(at 184.15 114.3 0)
 		(fields_autoplaced yes)
 		(effects
@@
 				(size 1.27 1.27)
 			)
-			(justify right bottom)
+			(justify left bottom)
 		)
 	)
 	(label "SCLK_A"
-		(at 223.52 99.06 180)
+		(at 184.15 99.06 0)
 		(fields_autoplaced yes)
 		(effects
@@
 				(size 1.27 1.27)
 			)
-			(justify right bottom)
+			(justify left bottom)
 		)
 	)
@@
 	)
 	(label "MOSI_A"
-		(at 223.52 109.22 180)
+		(at 184.15 109.22 0)
 		(fields_autoplaced yes)
 		(effects
@@
 				(size 1.27 1.27)
 			)
-			(justify right bottom)
+			(justify left bottom)
 		)
 	)
@@
 	(hierarchical_label "MOSI"
 		(shape input)
-		(at 190.5 109.22 180)
+		(at 217.17 109.22 0)
 		(fields_autoplaced yes)
 		(effects
@@
 				(size 1.27 1.27)
 			)
-			(justify right)
+			(justify left)
 		)
 	)
 	(hierarchical_label "CS_"
 		(shape input)
-		(at 190.5 104.14 180)
+		(at 217.17 104.14 0)
 		(fields_autoplaced yes)
 		(effects
@@
 				(size 1.27 1.27)
 			)
-			(justify right)
+			(justify left)
 		)
 	)
 	(hierarchical_label "SCLK"
 		(shape input)
-		(at 190.5 99.06 180)
+		(at 217.17 99.06 0)
 		(fields_autoplaced yes)
 		(effects
@@
 				(size 1.27 1.27)
 			)
-			(justify right)
+			(justify left)
 		)
 	)
 	(hierarchical_label "MISO"
 		(shape output)
-		(at 190.5 114.3 180)
+		(at 217.17 114.3 0)
 		(fields_autoplaced yes)
 		(effects
@@
 				(size 1.27 1.27)
 			)
-			(justify right)
+			(justify left)
 		)
 	)
 	(symbol
 		(lib_id "Power_Port:5VA")
-		(at 218.44 88.9 0)
+		(at 189.23 88.9 0)
+		(mirror y)
 		(unit 1)
 		(exclude_from_sim no)
@@
 		(fields_autoplaced yes)
 		(property "Reference" "#PWR0420"
-			(at 218.44 92.71 0)
+			(at 189.23 92.71 0)
 			(effects
 				(font
@@
 		)
 		(property "Value" "5VA"
-			(at 218.44 83.82 0)
+			(at 189.23 83.82 0)
 			(effects
 				(font
@@
 		)
 		(property "Footprint" ""
-			(at 218.44 88.9 0)
+			(at 189.23 88.9 0)
 			(effects
 				(font
@@
 		)
 		(property "Datasheet" ""
-			(at 218.44 88.9 0)
+			(at 189.23 88.9 0)
 			(effects
 				(font
@@
 		)
 		(property "Description" ""
-			(at 218.44 88.9 0)
+			(at 189.23 88.9 0)
 			(effects
 				(font
@@
 	(symbol
 		(lib_id "Power_Port:GNDA")
-		(at 228.6 96.52 0)
+		(at 179.07 96.52 0)
+		(mirror y)
 		(unit 1)
 		(exclude_from_sim no)
@@
 		(dnp no)
 		(property "Reference" "#PWR0422"
-			(at 228.6 100.838 0)
+			(at 179.07 100.838 0)
 			(effects
 				(font
@@
 		)
 		(property "Value" "GNDA"
-			(at 228.6 99.06 0)
+			(at 179.07 99.06 0)
 			(effects
 				(font
@@
 		)
 		(property "Footprint" ""
-			(at 228.6 93.98 0)
+			(at 179.07 93.98 0)
 			(effects
 				(font
@@
 		)
 		(property "Datasheet" ""
-			(at 228.092 98.806 0)
+			(at 179.578 98.806 0)
 			(effects
 				(font
@@
 		)
 		(property "Description" ""
-			(at 228.6 96.52 0)
+			(at 179.07 96.52 0)
 			(effects
 				(font
@@
 	(symbol
 		(lib_id "Power_Port:GNDA")
-		(at 215.9 127 0)
+		(at 191.77 127 0)
+		(mirror y)
 		(unit 1)
 		(exclude_from_sim no)
@@
 		(dnp no)
 		(property "Reference" "#PWR0430"
-			(at 215.9 131.318 0)
+			(at 191.77 131.318 0)
 			(effects
 				(font
@@
 		)
 		(property "Value" "GNDA"
-			(at 215.9 129.54 0)
+			(at 191.77 129.54 0)
 			(effects
 				(font
@@
 		)
 		(property "Footprint" ""
-			(at 215.9 124.46 0)
+			(at 191.77 124.46 0)
 			(effects
 				(font
@@
 		)
 		(property "Datasheet" ""
-			(at 215.392 129.286 0)
+			(at 192.278 129.286 0)
 			(effects
 				(font
@@
 		)
 		(property "Description" ""
-			(at 215.9 127 0)
+			(at 191.77 127 0)
 			(effects
 				(font
@@
 	(symbol
 		(lib_id "Power_Port:VDD")
-		(at 189.23 88.9 0)
+		(at 218.44 88.9 0)
+		(mirror y)
 		(unit 1)
 		(exclude_from_sim no)
@@
 		(fields_autoplaced yes)
 		(property "Reference" "#PWR0419"
-			(at 189.23 92.71 0)
+			(at 218.44 92.71 0)
 			(effects
 				(font
@@
 		)
 		(property "Value" "VDD"
-			(at 189.23 83.82 0)
+			(at 218.44 83.82 0)
 			(effects
 				(font
@@
 		)
 		(property "Footprint" ""
-			(at 189.23 88.9 0)
+			(at 218.44 88.9 0)
 			(effects
 				(font
@@
 		)
 		(property "Datasheet" ""
-			(at 189.23 92.71 0)
+			(at 218.44 92.71 0)
 			(effects
 				(font
@@
 		)
 		(property "Description" ""
-			(at 189.23 88.9 0)
+			(at 218.44 88.9 0)
 			(effects
 				(font
@@
 	(symbol
 		(lib_id "Power_Port:GNDB")
-		(at 179.07 96.52 0)
+		(at 228.6 96.52 0)
+		(mirror y)
 		(unit 1)
 		(exclude_from_sim no)
@@
 		(dnp no)
 		(property "Reference" "#PWR0421"
-			(at 179.07 100.838 0)
+			(at 228.6 100.838 0)
 			(effects
 				(font
@@
 		)
 		(property "Value" "GNDB"
-			(at 179.07 99.06 0)
+			(at 228.6 99.06 0)
 			(effects
 				(font
@@
 		)
 		(property "Footprint" ""
-			(at 179.07 93.98 0)
+			(at 228.6 93.98 0)
 			(effects
 				(font
@@
 		)
 		(property "Datasheet" ""
-			(at 178.562 98.806 0)
+			(at 229.108 98.806 0)
 			(effects
 				(font
@@
 		)
 		(property "Description" ""
-			(at 179.07 96.52 0)
+			(at 228.6 96.52 0)
 			(effects
 				(font
@@
 	(symbol
 		(lib_id "Power_Port:GNDB")
-		(at 190.5 127 0)
+		(at 217.17 127 0)
+		(mirror y)
 		(unit 1)
 		(exclude_from_sim no)
@@
 		(dnp no)
 		(property "Reference" "#PWR0429"
-			(at 190.5 131.318 0)
+			(at 217.17 131.318 0)
 			(effects
 				(font
@@
 		)
 		(property "Value" "GNDB"
-			(at 190.5 129.54 0)
+			(at 217.17 129.54 0)
 			(effects
 				(font
@@
 		)
 		(property "Footprint" ""
-			(at 190.5 124.46 0)
+			(at 217.17 124.46 0)
 			(effects
 				(font
@@
 		)
 		(property "Datasheet" ""
-			(at 189.992 129.286 0)
+			(at 217.678 129.286 0)
 			(effects
 				(font
@@
 		)
 		(property "Description" ""
-			(at 190.5 127 0)
+			(at 217.17 127 0)
 			(effects
 				(font
@@
 	(symbol
 		(lib_id "Isolators:ISO7341CQDWQ1")
-		(at 203.2 86.36 0)
+		(at 204.47 86.36 0)
+		(mirror y)
 		(unit 1)
 		(exclude_from_sim no)
@@
 		(on_board yes)
 		(dnp no)
-		(fields_autoplaced yes)
 		(property "Reference" "U404"
-			(at 203.2 82.55 0)
+			(at 204.47 82.55 0)
 			(effects
 				(font
@@
 		)
 		(property "Value" "ISO7341CQDWQ1"
-			(at 203.2 85.09 0)
+			(at 204.47 85.09 0)
 			(effects
 				(font
@@
 		)
 		(property "Footprint" "IC:SOIC-16-wide"
-			(at 203.2 86.36 0)
+			(at 204.47 86.36 0)
 			(effects
 				(font
@@
 		)
 		(property "Datasheet" "https://www.ti.com/lit/ds/symlink/iso7340-q1.pdf?HQS=dis-dk-null-digikeymode-dsf-pf-null-wwe&ts=1648920938853&ref_url=https%253A%252F%252Fwww.ti.com%252Fgeneral%252Fdocs%252Fsuppproductinfo.tsp%253FdistId%253D10%2526gotoUrl%253Dhttps%253A%252F%252Fwww.ti.com%252Flit%252Fgpn%252Fiso7340-q1"
-			(at 203.2 86.36 0)
+			(at 204.47 86.36 0)
 			(effects
 				(font
@@
 		)
 		(property "Description" "General Purpose Digital Isolator 3000Vrms 4 Channel 25Mbps 25kV/µs CMTI 16-SOIC (0.295\", 7.50mm Width)"
-			(at 203.2 86.36 0)
+			(at 204.47 86.36 0)
 			(effects
 				(font

Commit message: update
Connections:
- net SCLK renamed SCL_5VK
- net SCLK_A renamed SCL_5VK_A
Changed lines of the file:
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@@
 		)
 	)
-	(label "SCLK_A"
+	(label "SCL_5VK_A"
 		(at 181.61 69.85 0)
 		(fields_autoplaced yes)
@@
 		)
 	)
-	(label "SCLK_A"
+	(label "SCL_5VK_A"
 		(at 184.15 99.06 0)
 		(fields_autoplaced yes)
@@
 		)
 	)
-	(hierarchical_label "SCLK"
+	(hierarchical_label "SCL_5VK"
 		(shape input)
 		(at 217.17 99.06 0)
@@
 		(dnp no)
 		(fields_autoplaced yes)
-		(property "Reference" "#PWR0420"
+		(property "Reference" "#PWR0419"
 			(at 189.23 92.71 0)
 			(effects
@@
 			(project "SACE-HW"
 				(path "/4c1e5ca8-aa0f-4a8e-bffe-6765adb2e3e8/bda9c1af-9e39-4d1c-9beb-c58cbb11e7a4"
-					(reference "#PWR0420")
+					(reference "#PWR0419")
 					(unit 1)
 				)
@@
 		(on_board yes)
 		(dnp no)
-		(property "Reference" "#PWR0422"
+		(property "Reference" "#PWR0421"
 			(at 179.07 100.838 0)
 			(effects
@@
 			(project "SACE-HW"
 				(path "/4c1e5ca8-aa0f-4a8e-bffe-6765adb2e3e8/bda9c1af-9e39-4d1c-9beb-c58cbb11e7a4"
-					(reference "#PWR0422")
+					(reference "#PWR0421")
 					(unit 1)
 				)
@@
 		(on_board yes)
 		(dnp no)
-		(property "Reference" "#PWR0430"
+		(property "Reference" "#PWR0429"
 			(at 191.77 131.318 0)
 			(effects
@@
 			(project "SACE-HW"
 				(path "/4c1e5ca8-aa0f-4a8e-bffe-6765adb2e3e8/bda9c1af-9e39-4d1c-9beb-c58cbb11e7a4"
-					(reference "#PWR0430")
+					(reference "#PWR0429")
 					(unit 1)
 				)
@@
 		(dnp no)
 		(fields_autoplaced yes)
-		(property "Reference" "#PWR0419"
+		(property "Reference" "#PWR0420"
 			(at 218.44 92.71 0)
 			(effects
@@
 			(project "SACE-HW"
 				(path "/4c1e5ca8-aa0f-4a8e-bffe-6765adb2e3e8/bda9c1af-9e39-4d1c-9beb-c58cbb11e7a4"
-					(reference "#PWR0419")
+					(reference "#PWR0420")
 					(unit 1)
 				)
@@
 		(on_board yes)
 		(dnp no)
-		(property "Reference" "#PWR0421"
+		(property "Reference" "#PWR0422"
 			(at 228.6 100.838 0)
 			(effects
@@
 			(project "SACE-HW"
 				(path "/4c1e5ca8-aa0f-4a8e-bffe-6765adb2e3e8/bda9c1af-9e39-4d1c-9beb-c58cbb11e7a4"
-					(reference "#PWR0421")
+					(reference "#PWR0422")
 					(unit 1)
 				)
@@
 		(on_board yes)
 		(dnp no)
-		(property "Reference" "#PWR0429"
+		(property "Reference" "#PWR0430"
 			(at 217.17 131.318 0)
 			(effects
@@
 			(project "SACE-HW"
 				(path "/4c1e5ca8-aa0f-4a8e-bffe-6765adb2e3e8/bda9c1af-9e39-4d1c-9beb-c58cbb11e7a4"
-					(reference "#PWR0429")
+					(reference "#PWR0430")
 					(unit 1)
 				)
