File: I2C.kicad_sch (KiCad schematic)
At the start: 29 parts, among them J601 2350514-8, J602 XH-4A connector, J603 XH-4A connector, J604 2350514-8, J605 2350514-8, U601 MCP4728T-E_UN, U602 TLV9302IDR, U603 TLA2528IRTER, U604 TLA2528IRTER

Commit message: update
Parts:
- removed C606, C607, C608: 885012107015, Capacitors:C0603, symbol Capacitors:885012106022
- removed J604, J605: 2350514-8, Connectors:CONN8_2350514-8_TEC, symbol Connectors:2350514-8
- removed R611: RC0805JR-070RL, Resistors:R0805, symbol Resistors:RC0805JR-07100KL
- removed R612: RC0805JR-070RL, Resistors:R0603, symbol Resistors:RC0805JR-070RL
- removed U604: TLA2528IRTER, QFN50P300X300X80-17N-D, symbol ADC:TLA2528IRTER
- added C505, C507: 885012107015, Capacitors:C0805, symbol Capacitors:885012107015
- added J504, J505: 2350514-8, Connectors:CONN8_2350514-8_TEC, symbol Connectors:2350514-8
- added R503, R504: RC0805JR-074K7L, Resistors:R0805, symbol Resistors:RC0805JR-074K7L
- added R513: RC0805JR-0710KL, Resistors:R0805, symbol Resistors:RC0805JR-0710KL
- added U504: TCA9617BDGKR, IC:SOP65P490X110-8N, symbol Interface:TCA9617BDGKR
- C501: renamed from C601; footprint Capacitors:C0603 -> Capacitors:C0805; symbol Capacitors:885012106022 -> Capacitors:885012107015; Manufacturer Part Number 885012106022 -> 885012107015; Supplier Part Number 732-7919-1-ND -> 732-7625-1-ND
- C502: renamed from C602; footprint Capacitors:C0603 -> Capacitors:C0805; symbol Capacitors:885012106022 -> Capacitors:885012107015; Manufacturer Part Number 885012106022 -> 885012107015; Supplier Part Number 732-7919-1-ND -> 732-7625-1-ND
- C503: renamed from C603; footprint Capacitors:C0603 -> Capacitors:C0805; symbol Capacitors:885012106022 -> Capacitors:885012107015; Manufacturer Part Number 885012106022 -> 885012107015; Supplier Part Number 732-7919-1-ND -> 732-7625-1-ND
- C504: renamed from C604; footprint Capacitors:C0603 -> Capacitors:C0805; symbol Capacitors:885012106022 -> Capacitors:885012107015; Manufacturer Part Number 885012106022 -> 885012107015; Supplier Part Number 732-7919-1-ND -> 732-7625-1-ND
- C506: renamed from C605; footprint Capacitors:C0603 -> Capacitors:C0805; symbol Capacitors:885012106022 -> Capacitors:885012107015; Manufacturer Part Number 885012106022 -> 885012107015; Supplier Part Number 732-7919-1-ND -> 732-7625-1-ND
- R506: renamed from R604; value RC0805JR-070RL -> 0hms_0.5W; footprint Resistors:R0603 -> Resistors:R0805; symbol Resistors:RC0805JR-070RL -> Resistors:0hms_0.5W; Manufacturer Yageo -> Keystone Electronics; Manufacturer Part Number RC0805JR-070RL -> 5106; Puissance (Watts) 1/8W -> 1/2W; Supplier Part Number 311-0.0ARCT-ND -> 36-5106CT-ND; Supplier_1 (none) -> Digikey
- R509: renamed from R607; value RC0805JR-070RL -> 0hms_0.5W; footprint Resistors:R0603 -> Resistors:R0805; symbol Resistors:RC0805JR-070RL -> Resistors:0hms_0.5W; Manufacturer Yageo -> Keystone Electronics; Manufacturer Part Number RC0805JR-070RL -> 5106; Puissance (Watts) 1/8W -> 1/2W; Supplier Part Number 311-0.0ARCT-ND -> 36-5106CT-ND; Supplier_1 (none) -> Digikey
- renumbered J601 to J501, J602 to J502, J603 to J503, R601 to R501, R602 to R502, R603 to R505, R605 to R507, R606 to R508, R608 to R510, R609 to R511, R610 to R512, U601 to U501, U602 to U502, U603 to U503
Connections:
- net 5VB: now also R513.1, U504.8 (VCCB)
- net GNDB: now also J501.2, J501.4, C505.1, C507.1, J504.2, J504.4, J504.6, J504.8, J505.2, J505.4, J505.6, J505.8, U504.4 (GND); no longer J501.5, J501.7
- net OUTA_10V: now also C505.2
- net OUTB_10V: now also J501.3, C507.2; no longer J501.2
- net OUTC: now also J501.5; no longer J501.3
- net OUTD: now also J501.7; no longer J501.4
- net SCL: now also R503.1, U504.2 (SCLA); no longer J502.3, J503.3, R501.1, U501.2 (SCL), U503.13 (SCL)
- net SDA: now also R504.1, U504.3 (SDAA); no longer J502.2, J503.2, R502.1, U501.3 (SDA), U503.14 (SDA)
- net GPIO2: now reaches U503.1 (AIN2/GPIO2)
- net GPIO2: now also J504.5
- net GPIO0: now reaches U503.15 (AIN0/GPIO0)
- net GPIO0: now also J504.1
- net GPIO1: now reaches U503.16 (AIN1/GPIO1)
- net GPIO1: now also J504.3
- net GPIO3: now reaches U503.2 (AIN3/GPIO3)
- net GPIO3: now also J504.7
- net GPIO4: now reaches U503.3 (AIN4/GPIO4)
- net GPIO4: now also J505.1
- net GPIO5: now reaches U503.4 (AIN5/GPIO5)
- net GPIO5: now also J505.3
- net GPIO6: now reaches U503.5 (AIN6/GPIO6)
- net GPIO6: now also J505.5
- net GPIO7: now reaches U503.6 (AIN7/GPIO7)
- net GPIO7: now also J505.7
- new net: R513.2, U504.5 (EN)
- new net SCL_5V: J502.3, J503.3, R501.1, U501.2 (SCL), U503.13 (SCL), U504.7 (SCLB)
- new net SDA_5V: J502.2, J503.2, R502.1, U501.3 (SDA), U503.14 (SDA), U504.6 (SDAB)
- new net VDD: R503.2, R504.2, U504.1 (VCCA)
Other:
- note removed: "Current addr: 0x14 (Check P.15 datasheet)"
- moved on the sheet: C501, C502, C503, C504, C506, J501, J502, J503, R501, R502, R505, R506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
