File: LV_PSU.kicad_sch (KiCad schematic)
At the start: 31 parts, among them IC1 1769205241, J1 1935161, J2 2350514-8, J3 Header_Male_Pin_2.54mm_1X2_,_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, U1 OKI-78SR-5_1.5-W36H-C, U2 AZ1117IH-3.3TRG1, U3 AZ1117IH-3.3TRG1

Commit message: finalisation de la schématique
Parts:
- added F201: 39511000440, Fuses:TE5_395, symbol Fuses:39511000440
- F202: renamed from F1; Current Rating (A) 500 mA -> 1A; Description_1 (none) -> FUSE BOARD MNT 1A 125VAC RADIAL; Description_2 (none) -> FUSE HOLDER RADIAL 250V 6.3A PCB; Manufacturer Part Number 56200001009 -> 39511000440; Manufacturer Part Number_1 (none) -> 56200001009; Manufacturer_1 (none) -> Littelfuse Inc.; Supplier Part Number WK0009-ND -> WK4348BK-ND; Supplier Part Number_1 (none) -> WK0009-ND; Supplier_1 (none) -> Digikey
- renumbered C5 to C201, C3 to C202, C6 to C203, C1 to C204, C2 to C205, C4 to C206, D2 to D201, D4 to D202, D1 to D203, D3 to D204, D5 to D205, IC1 to IC201, J3 to J201, J1 to J202, J2 to J203, R2 to R201, R4 to R202, R1 to R203, R3 to R204, R5 to R205, TP5 to TP201, TP3 to TP202, TP6 to TP203, TP7 to TP204, TP1 to TP205, TP4 to TP206, TP2 to TP207, U2 to U201, U1 to U202, U3 to U203
Connections:
- net 12VB: now also C204.2, F202.2, R203.2, TP205.1 (TP), U202.1 (Vin); no longer F202.1, J202.2
- net 5VA: now also F201.2; no longer IC201.5 (+VOUT)
- new net: F201.1, IC201.5 (+VOUT)
- new net: F202.1, J202.2
Other:
- moved on the sheet: F202

Commit message: update
Parts:
- removed TP201, TP202, TP203, TP204, TP205, TP206, TP207: Test_Point_THM, Connectors:Keystone_5001, symbol Connectors:Test_Point_THM
Other:
- note removed: "12V IN"
