File: MCU.kicad_sch (KiCad schematic)
At the start: 37 parts, among them J1 XH-4A connector, J2 Header_Male_Pin_2.54mm_1X6_,_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, SW1 PTS645SM43SMTR92, SW2 PTS645SM43SMTR92, U1 STM32F446RE

Commit message: update schematic
Other:
- note added: "HSE AND LSE need to be routed as close as possible to the mcu. Check AN2867"
- note removed: "HSE AND LSE need to be routed as close as possible to the mcu. See : AN2867"
- moved on the sheet: C14, J2, R12, R13, SW2

Commit message: update schematic
Parts:
- renumbered C10 to C301, C4 to C302, C7 to C303, C8 to C304, C1 to C305, C3 to C306, C13 to C307, C5 to C308, C6 to C309, C14 to C310, C2 to C311, C11 to C312, C12 to C313, C9 to C314, D1 to D301, D2 to D302, D3 to D303, J2 to J301, J1 to J302, R10 to R301, R7 to R302, R2 to R303, R13 to R304, R1 to R305, R12 to R306, R3 to R307, R5 to R308, R4 to R309, R8 to R310, R9 to R311, R11 to R312, R6 to R313, SW2 to SW301, SW1 to SW302, U1 to U301, XTAL2 to XTAL301, XTAL1 to XTAL302

Commit message: update schematique
Parts:
- renumbered C311 to C10, C306 to C11, C302 to C12, C308 to C13, C309 to C14, C303 to C15, C304 to C16, C314 to C17, C301 to C18, C312 to C19, C313 to C20, C307 to C21, C310 to C22, C305 to C9, D301 to D7, D302 to D8, D303 to D9, J302 to J4, J301 to J5, R309 to R10, R308 to R11, R313 to R12, R302 to R13, R310 to R14, R311 to R15, R301 to R16, R312 to R17, R306 to R18, R304 to R19, R305 to R7, R303 to R8, R307 to R9, SW302 to SW1, SW301 to SW2, U301 to U5, XTAL302 to XTAL1, XTAL301 to XTAL2

Commit message: update schematique
Parts:
- removed R12: RC0805JR-072K2L, Resistors:R0805, symbol Resistors:RC0805JR-072K2L
- renumbered C18 to C301, C12 to C302, C15 to C303, C16 to C304, C9 to C305, C11 to C306, C21 to C307, C13 to C308, C14 to C309, C22 to C310, C10 to C311, C19 to C312, C20 to C313, C17 to C314, D7 to D301, D8 to D302, D9 to D303, J5 to J301, J4 to J302, R16 to R301, R13 to R302, R8 to R303, R19 to R304, R7 to R305, R18 to R306, R9 to R307, R11 to R308, R10 to R309, R14 to R310, R15 to R311, R17 to R312, SW2 to SW301, SW1 to SW302, U5 to U301, XTAL2 to XTAL301, XTAL1 to XTAL302
Other:
- moved on the sheet: R309

Commit message: update schematic
Parts:
- renumbered C302 to C10, C308 to C11, C309 to C12, C303 to C13, C304 to C14, C314 to C15, C301 to C16, C312 to C17, C313 to C18, C307 to C19, C310 to C20, C305 to C7, C311 to C8, C306 to C9, D301 to D6, D302 to D7, D303 to D8, J302 to J4, J301 to J5, R309 to R10, R302 to R11, R310 to R12, R311 to R13, R301 to R14, R312 to R15, R306 to R16, R304 to R17, R305 to R6, R303 to R7, R307 to R8, R308 to R9, SW302 to SW1, SW301 to SW2, U301 to U4, XTAL302 to XTAL1, XTAL301 to XTAL2
Connections:
- net DGND renamed GNDB

Commit message: finalisation de la schématique
Parts:
- renumbered C16 to C301, C10 to C302, C13 to C303, C14 to C304, C7 to C305, C9 to C306, C19 to C307, C11 to C308, C12 to C309, C20 to C310, C8 to C311, C17 to C312, C18 to C313, C15 to C314, D6 to D301, D7 to D302, D8 to D303, J5 to J301, J4 to J302, R14 to R301, R11 to R302, R7 to R303, R17 to R304, R6 to R305, R16 to R306, R8 to R307, R9 to R308, R10 to R309, R12 to R310, R13 to R311, R15 to R312, SW2 to SW301, SW1 to SW302, U4 to U301, XTAL2 to XTAL301, XTAL1 to XTAL302
Connections:
- net 5V renamed 5VB

Commit message: clean up
Parts:
- removed C301, C307, C311, C313, C314: 885012207098, Capacitors:C0805, symbol Capacitors:885012207098
- removed C302, C303: 885012007027, Capacitors:C0805, symbol Capacitors:885012007027
- removed C304, C308: 885012107015, Capacitors:C0805, symbol Capacitors:885012107015
- removed C305, C306: 885012007053, Capacitors:C0805, symbol Capacitors:885012007053
- removed C309: 885012207092, Capacitors:C0805, symbol Capacitors:885012207092
- removed C312: 885012107018, Capacitors:C0805, symbol Capacitors:885012107018
- removed J301: Header_Male_Pin_2.54mm_1X6_,_Unshrouded, Connectors:Headers_2.54mm_1X6, symbol Connectors:Header_Male_Pin_2.54mm_1X6_,_Unshrouded
- removed J302: XH-4A connector, Connectors:XH-4A, symbol Connectors:XH-4A connector
- removed R301: RC0805JR-0710KL, Resistors:R0805, symbol Resistors:RC0805JR-0710KL
- removed R302, R303: RC0805JR-070RL, Resistors:R0805, symbol Resistors:RC0805JR-070RL
- removed R305: RC0805JR-074K7L, Resistors:R0805, symbol Resistors:RC0805JR-074K7L
- removed R307: RC0805JR-07150RL, Resistors:R0805, symbol Resistors:RC0805JR-07150RL
- removed R308, R309: RC0805JR-07470RL, Resistors:R0805, symbol Resistors:RC0805JR-07470RL
- removed SW302: PTS645SM43SMTR92, Switches:PTS645_6X6X4_SMD, symbol Switches:PTS645SM43SMTR92
- removed U301: STM32F446RE, IC:LQFP-64, symbol STMicroelectronics:STM32F446RE
- removed XTAL301: ABS25-32.768KHZ-6-T, Crystals:ABS25, symbol Crystals:ABS25-32.768KHZ-6-T
- removed XTAL302: 7A-8.000MAHJ-T, Crystals:TXC_7A_Series, symbol Crystals:7A-8.000MAHJ-T
Connections:
- net PA5 renamed BLINK
- net PA6 renamed DEBUG
- net PA7 renamed ERROR
- no-connect marks 4 -> 2
Other:
- note removed: "HSE"
- note removed: "HSE AND LSE need to be routed as close as possible to the mcu. Check AN2867"
- note removed: "LSE"
- note removed: "RESET"
- note removed: "SWD Connector"
- note removed: "USART2 - DEBUG (5V LOGIC)"

Commit message: update
Parts:
- added U301: ESP32-DEVKITC-32D, Assembly:MODULE_ESP32-DEVKITC-32D, symbol Boards:ESP32-DEVKITC-32D
- renumbered C310 to C301, R304 to R301, R306 to R302, R310 to R303, R311 to R304, R312 to R305
Connections:
- net GNDB: now also U301.J2-14 (GND1), U301.J3-1 (GND3), U301.J3-7 (GND2)
- net VDD: now also U301.J2-1 (3V3), U301.J2-2 (EN)
- net BLINK renamed IO2
- net IO2: now also U301.J3-15 (IO2)
- net DEBUG renamed IO3
- net IO3: now also U301.J3-5 (IO3)
- net ERROR renamed IO25
- net IO25: now also U301.J2-9 (IO25)
- net USER_BTN renamed IO26
- net IO26: now also U301.J2-10 (IO26)
- new net IO0: U301.J3-14 (IO0)
- new net IO1: U301.J3-4 (IO1)
- new net IO10: U301.J2-17 (IO10)
- new net IO11: U301.J2-18 (IO11)
- new net IO12: U301.J2-13 (IO12)
- new net IO13: U301.J2-15 (IO13)
- new net IO14: U301.J2-12 (IO14)
- new net IO15: U301.J3-16 (IO15)
- new net IO16: U301.J3-12 (IO16)
- new net IO17: U301.J3-11 (IO17)
- new net IO18: U301.J3-9 (IO18)
- new net IO19: U301.J3-8 (IO19)
- new net IO21: U301.J3-6 (IO21)
- new net IO22: U301.J3-3 (IO22)
- new net IO23: U301.J3-2 (IO23)
- new net IO27: U301.J2-11 (IO27)
- new net IO32: U301.J2-7 (IO32)
- new net IO33: U301.J2-8 (IO33)
- new net IO34: U301.J2-5 (IO34)
- new net IO35: U301.J2-6 (IO35)
- new net IO36: U301.J2-3 (IO36)
- new net IO39: U301.J2-4 (IO39)
- new net IO4: U301.J3-13 (IO4)
- new net IO5: U301.J3-10 (IO5)
- new net IO6: U301.J3-19 (IO6)
- new net IO7: U301.J3-18 (IO7)
- new net IO8: U301.J3-17 (IO8)
- new net IO9: U301.J2-16 (IO9)
Other:
- moved on the sheet: C301, D301, D302, D303, R301, R302, R303, R304, R305, SW301
