File: SACE-HW.kicad_sch (KiCad schematic)
At the start: 8 parts, among them J101 Header_Male_Pin_2.54mm_1X5_,_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

Commit message: clean up
Other:
- removed sheet USB_Serial
- sheet SD_CARD ports: added CARD_CS; removed CARD_CK, CARD_CMD, CARD_CS/DAT3, CARD_D0, CARD_DAT1, CARD_DAT2
- moved on the sheet: C101, J101, R101, R102

Commit message: update
Parts:
- removed C101: 885012207098, Capacitors:C0805, symbol Capacitors:885012207098
- removed J101: Header_Male_Pin_2.54mm_1X5_,_Unshrouded, Connectors:Headers_2.54mm_1X5, symbol Connectors:Header_Male_Pin_2.54mm_1X5_,_Unshrouded
- removed R101: RC0805JR-074K7L, Resistors:R0805, symbol Resistors:RC0805JR-074K7L
- removed R102: RC0805JR-07150RL, Resistors:R0805, symbol Resistors:RC0805JR-07150RL
- added J101: 2350514-8, Connectors:CONN8_2350514-8_TEC, symbol Connectors:2350514-8
Connections:
- net GNDB: now also J101.2, J101.4, J101.6, J101.8
- new net IO0: J101.1
- new net IO1: J101.3
- new net IO32: J101.5
- new net IO33: J101.7
- no-connect marks 8 -> 9
Other:
- sheet HV ports: added SCL_5VK; removed SCLK
- sheet I2C ports: added SCL_5V, SDA_5V; removed SCL, SDA
- sheet MCU ports: added IO0, IO1, IO10, IO11, IO12, IO13, IO14, IO15, IO16, IO17, IO18, IO19, IO2, IO21, IO22, IO23, IO25, IO26, IO27, IO3, IO32, IO33, IO34, IO35, IO36, IO39, IO4, IO5, IO6, IO7, IO8, IO9; removed NRST, PA0, PA1, PA10, PA11, PA12, PA15, PA4, PA5, PA6, PA7, PA8, PA9, PB0, PB1, PB10, PB12, PB13, PB14, PB15, PB2, PB4, PB5, PB6, PB7, PB8, PB9, PC0, PC1, PC10, PC11, PC12, PC2, PC3, PC4, PC5, PC6, PC7, PC8, PC9, PD2, USART2_RX, USART2_TX, VBat
