File: SD_CARD.kicad_sch (KiCad schematic)
At the start: 17 parts, among them J801 MEM2075-00-140-01-A

Commit message: update schematic
Parts:
- renumbered C803 to C40, C801 to C41, C802 to C42, J801 to J18, R803 to R46, R804 to R47, R805 to R48, R806 to R49, R807 to R50, R802 to R51, R801 to R52, SB801 to SB3, SB803 to SB4, SB805 to SB5, SB802 to SB6, SB804 to SB7, SB806 to SB8
Connections:
- net DGND renamed GNDB
Changed lines of the file:
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@@
 		(on_board yes)
 		(dnp yes)
-		(property "Reference" "R803"
+		(property "Reference" "R46"
 			(at 95.25 106.68 0)
 			(effects
@@
 			(project "SACE-HW"
 				(path "/4c1e5ca8-aa0f-4a8e-bffe-6765adb2e3e8/6b453246-6ae6-4c73-99ea-9f79a5f14ff1"
-					(reference "R803")
+					(reference "R46")
 					(unit 1)
 				)
@@
 		(on_board yes)
 		(dnp yes)
-		(property "Reference" "R805"
+		(property "Reference" "R48"
 			(at 95.25 124.46 0)
 			(effects
@@
 			(project "SACE-HW"
 				(path "/4c1e5ca8-aa0f-4a8e-bffe-6765adb2e3e8/6b453246-6ae6-4c73-99ea-9f79a5f14ff1"
-					(reference "R805")
+					(reference "R48")
 					(unit 1)
 				)
@@
 		(dnp no)
 		(fields_autoplaced yes)
-		(property "Reference" "SB801"
+		(property "Reference" "SB3"
 			(at 156.21 97.79 0)
 			(effects
@@
 			(project "SACE-HW"
 				(path "/4c1e5ca8-aa0f-4a8e-bffe-6765adb2e3e8/6b453246-6ae6-4c73-99ea-9f79a5f14ff1"
-					(reference "SB801")
+					(reference "SB3")
 					(unit 1)
 				)
@@
 		(on_board yes)
 		(dnp no)
-		(property "Reference" "C802"
+		(property "Reference" "C42"
 			(at 187.325 59.69 90)
 			(effects
@@
 			(project "SACE-HW"
 				(path "/4c1e5ca8-aa0f-4a8e-bffe-6765adb2e3e8/6b453246-6ae6-4c73-99ea-9f79a5f14ff1"
-					(reference "C802")
+					(reference "C42")
 					(unit 1)
 				)
@@
 		(dnp no)
 		(fields_autoplaced yes)
-		(property "Reference" "R801"
+		(property "Reference" "R52"
 			(at 144.78 63.5 90)
 			(effects
@@
 			(project "SACE-HW"
 				(path "/4c1e5ca8-aa0f-4a8e-bffe-6765adb2e3e8/6b453246-6ae6-4c73-99ea-9f79a5f14ff1"
-					(reference "R801")
+					(reference "R52")
 					(unit 1)
 				)
@@
 		(dnp no)
 		(fields_autoplaced yes)
-		(property "Reference" "SB803"
+		(property "Reference" "SB4"
 			(at 156.21 106.68 0)
 			(effects
@@
 			(project "SACE-HW"
 				(path "/4c1e5ca8-aa0f-4a8e-bffe-6765adb2e3e8/6b453246-6ae6-4c73-99ea-9f79a5f14ff1"
-					(reference "SB803")
+					(reference "SB4")
 					(unit 1)
 				)
@@
 		(dnp no)
 		(fields_autoplaced yes)
-		(property "Reference" "J801"
+		(property "Reference" "J18"
 			(at 107.95 57.15 0)
 			(effects
@@
 			(project "SACE-HW"
 				(path "/4c1e5ca8-aa0f-4a8e-bffe-6765adb2e3e8/6b453246-6ae6-4c73-99ea-9f79a5f14ff1"
-					(reference "J801")
+					(reference "J18")
 					(unit 1)
 				)
@@
 		(dnp no)
 		(fields_autoplaced yes)
-		(property "Reference" "SB804"
+		(property "Reference" "SB7"
 			(at 175.26 106.68 0)
 			(effects
@@
 			(project "SACE-HW"
 				(path "/4c1e5ca8-aa0f-4a8e-bffe-6765adb2e3e8/6b453246-6ae6-4c73-99ea-9f79a5f14ff1"
-					(reference "SB804")
+					(reference "SB7")
 					(unit 1)
 				)
@@
 		(dnp no)
 		(fields_autoplaced yes)
-		(property "Reference" "SB806"
+		(property "Reference" "SB8"
 			(at 175.26 115.57 0)
 			(effects
@@
 			(project "SACE-HW"
 				(path "/4c1e5ca8-aa0f-4a8e-bffe-6765adb2e3e8/6b453246-6ae6-4c73-99ea-9f79a5f14ff1"
-					(reference "SB806")
+					(reference "SB8")
 					(unit 1)
 				)
@@
 		(on_board yes)
 		(dnp yes)
-		(property "Reference" "R804"
+		(property "Reference" "R47"
 			(at 95.25 115.57 0)
 			(effects
@@
 			(project "SACE-HW"
 				(path "/4c1e5ca8-aa0f-4a8e-bffe-6765adb2e3e8/6b453246-6ae6-4c73-99ea-9f79a5f14ff1"
-					(reference "R804")
+					(reference "R47")
 					(unit 1)
 				)
@@
 	)
 	(symbol
-		(lib_id "Power_Port:DGND")
+		(lib_id "Power_Port:GNDB")
 		(at 172.72 69.85 0)
 		(unit 1)
@@
 		(on_board yes)
 		(dnp no)
-		(property "Reference" "#PWR0803"
+		(property "Reference" "#PWR0136"
 			(at 172.72 74.168 0)
 			(effects
@@
 			)
 		)
-		(property "Value" "DGND"
-			(at 176.53 68.58 0)
+		(property "Value" "GNDB"
+			(at 172.72 72.39 0)
 			(effects
 				(font
@@
 			(project "SACE-HW"
 				(path "/4c1e5ca8-aa0f-4a8e-bffe-6765adb2e3e8/6b453246-6ae6-4c73-99ea-9f79a5f14ff1"
-					(reference "#PWR0803")
+					(reference "#PWR0136")
 					(unit 1)
 				)
@@
 		(dnp no)
 		(fields_autoplaced yes)
-		(property "Reference" "SB802"
+		(property "Reference" "SB6"
 			(at 175.26 97.79 0)
 			(effects
@@
 			(project "SACE-HW"
 				(path "/4c1e5ca8-aa0f-4a8e-bffe-6765adb2e3e8/6b453246-6ae6-4c73-99ea-9f79a5f14ff1"
-					(reference "SB802")
+					(reference "SB6")
 					(unit 1)
 				)
@@
 		(dnp no)
 		(fields_autoplaced yes)
-		(property "Reference" "R802"
+		(property "Reference" "R51"
 			(at 133.35 66.04 0)
 			(effects
@@
 			(project "SACE-HW"
 				(path "/4c1e5ca8-aa0f-4a8e-bffe-6765adb2e3e8/6b453246-6ae6-4c73-99ea-9f79a5f14ff1"
-					(reference "R802")
+					(reference "R51")
 					(unit 1)
 				)
@@
 		(on_board yes)
 		(dnp no)
-		(property "Reference" "C803"
+		(property "Reference" "C40"
 			(at 147.955 74.93 90)
 			(effects
@@
 			(project "SACE-HW"
 				(path "/4c1e5ca8-aa0f-4a8e-bffe-6765adb2e3e8/6b453246-6ae6-4c73-99ea-9f79a5f14ff1"
-					(reference "C803")
+					(reference "C40")
 					(unit 1)
 				)
@@
 		(dnp no)
 		(fields_autoplaced yes)
-		(property "Reference" "#PWR0801"
+		(property "Reference" "#PWR0134"
 			(at 142.24 58.42 0)
 			(effects
@@
 			(project "SACE-HW"
 				(path "/4c1e5ca8-aa0f-4a8e-bffe-6765adb2e3e8/6b453246-6ae6-4c73-99ea-9f79a5f14ff1"
-					(reference "#PWR0801")
+					(reference "#PWR0134")
 					(unit 1)
 				)
@@
 		(on_board yes)
 		(dnp yes)
-		(property "Reference" "R807"
+		(property "Reference" "R50"
 			(at 95.25 142.24 0)
 			(effects
@@
 			(project "SACE-HW"
 				(path "/4c1e5ca8-aa0f-4a8e-bffe-6765adb2e3e8/6b453246-6ae6-4c73-99ea-9f79a5f14ff1"
-					(reference "R807")
+					(reference "R50")
 					(unit 1)
 				)
@@
 	)
 	(symbol
-		(lib_id "Power_Port:DGND")
+		(lib_id "Power_Port:GNDB")
 		(at 129.54 85.09 0)
 		(unit 1)
@@
 		(on_board yes)
 		(dnp no)
-		(property "Reference" "#PWR0804"
+		(property "Reference" "#PWR0133"
 			(at 129.54 89.408 0)
 			(effects
@@
 			)
 		)
-		(property "Value" "DGND"
-			(at 133.35 83.82 0)
+		(property "Value" "GNDB"
+			(at 129.54 87.63 0)
 			(effects
 				(font
@@
 			(project "SACE-HW"
 				(path "/4c1e5ca8-aa0f-4a8e-bffe-6765adb2e3e8/6b453246-6ae6-4c73-99ea-9f79a5f14ff1"
-					(reference "#PWR0804")
+					(reference "#PWR0133")
 					(unit 1)
 				)
@@
 		(dnp no)
 		(fields_autoplaced yes)
-		(property "Reference" "#PWR0805"
+		(property "Reference" "#PWR0132"
 			(at 86.36 109.22 0)
 			(effects
@@
 			(project "SACE-HW"
 				(path "/4c1e5ca8-aa0f-4a8e-bffe-6765adb2e3e8/6b453246-6ae6-4c73-99ea-9f79a5f14ff1"
-					(reference "#PWR0805")
+					(reference "#PWR0132")
 					(unit 1)
 				)
@@
 		(on_board yes)
 		(dnp no)
-		(property "Reference" "C801"
+		(property "Reference" "C41"
 			(at 167.64 59.055 90)
 			(effects
@@
 			(project "SACE-HW"
 				(path "/4c1e5ca8-aa0f-4a8e-bffe-6765adb2e3e8/6b453246-6ae6-4c73-99ea-9f79a5f14ff1"
-					(reference "C801")
+					(reference "C41")
 					(unit 1)
 				)
@@
 		(dnp no)
 		(fields_autoplaced yes)
-		(property "Reference" "SB805"
+		(property "Reference" "SB5"
 			(at 156.21 115.57 0)
 			(effects
@@
 			(project "SACE-HW"
 				(path "/4c1e5ca8-aa0f-4a8e-bffe-6765adb2e3e8/6b453246-6ae6-4c73-99ea-9f79a5f14ff1"
-					(reference "SB805")
+					(reference "SB5")
 					(unit 1)
 				)
@@
 		(on_board yes)
 		(dnp yes)
-		(property "Reference" "R806"
+		(property "Reference" "R49"
 			(at 95.25 133.35 0)
 			(effects
@@
 			(project "SACE-HW"
 				(path "/4c1e5ca8-aa0f-4a8e-bffe-6765adb2e3e8/6b453246-6ae6-4c73-99ea-9f79a5f14ff1"
-					(reference "R806")
+					(reference "R49")
 					(unit 1)
 				)
@@
 		(dnp no)
 		(fields_autoplaced yes)
-		(property "Reference" "#PWR0802"
+		(property "Reference" "#PWR0135"
 			(at 172.72 58.42 0)
 			(effects
@@
 			(project "SACE-HW"
 				(path "/4c1e5ca8-aa0f-4a8e-bffe-6765adb2e3e8/6b453246-6ae6-4c73-99ea-9f79a5f14ff1"
-					(reference "#PWR0802")
+					(reference "#PWR0135")
 					(unit 1)
 				)

Commit message: finalisation de la schématique
Parts:
- renumbered C41 to C801, C42 to C802, C40 to C803, J18 to J801, R52 to R801, R51 to R802, R46 to R803, R47 to R804, R48 to R805, R49 to R806, R50 to R807, SB3 to SB801, SB6 to SB802, SB4 to SB803, SB7 to SB804, SB5 to SB805, SB8 to SB806
Changed lines of the file:
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@@
 		(on_board yes)
 		(dnp yes)
-		(property "Reference" "R46"
+		(property "Reference" "R803"
 			(at 95.25 106.68 0)
 			(effects
@@
 			(project "SACE-HW"
 				(path "/4c1e5ca8-aa0f-4a8e-bffe-6765adb2e3e8/6b453246-6ae6-4c73-99ea-9f79a5f14ff1"
-					(reference "R46")
+					(reference "R803")
 					(unit 1)
 				)
@@
 		(on_board yes)
 		(dnp yes)
-		(property "Reference" "R48"
+		(property "Reference" "R805"
 			(at 95.25 124.46 0)
 			(effects
@@
 			(project "SACE-HW"
 				(path "/4c1e5ca8-aa0f-4a8e-bffe-6765adb2e3e8/6b453246-6ae6-4c73-99ea-9f79a5f14ff1"
-					(reference "R48")
+					(reference "R805")
 					(unit 1)
 				)
@@
 		(dnp no)
 		(fields_autoplaced yes)
-		(property "Reference" "SB3"
+		(property "Reference" "SB801"
 			(at 156.21 97.79 0)
 			(effects
@@
 			(project "SACE-HW"
 				(path "/4c1e5ca8-aa0f-4a8e-bffe-6765adb2e3e8/6b453246-6ae6-4c73-99ea-9f79a5f14ff1"
-					(reference "SB3")
+					(reference "SB801")
 					(unit 1)
 				)
@@
 		(on_board yes)
 		(dnp no)
-		(property "Reference" "C42"
+		(property "Reference" "C802"
 			(at 187.325 59.69 90)
 			(effects
@@
 			(project "SACE-HW"
 				(path "/4c1e5ca8-aa0f-4a8e-bffe-6765adb2e3e8/6b453246-6ae6-4c73-99ea-9f79a5f14ff1"
-					(reference "C42")
+					(reference "C802")
 					(unit 1)
 				)
@@
 		(dnp no)
 		(fields_autoplaced yes)
-		(property "Reference" "R52"
+		(property "Reference" "R801"
 			(at 144.78 63.5 90)
 			(effects
@@
 			(project "SACE-HW"
 				(path "/4c1e5ca8-aa0f-4a8e-bffe-6765adb2e3e8/6b453246-6ae6-4c73-99ea-9f79a5f14ff1"
-					(reference "R52")
+					(reference "R801")
 					(unit 1)
 				)
@@
 		(dnp no)
 		(fields_autoplaced yes)
-		(property "Reference" "SB4"
+		(property "Reference" "SB803"
 			(at 156.21 106.68 0)
 			(effects
@@
 			(project "SACE-HW"
 				(path "/4c1e5ca8-aa0f-4a8e-bffe-6765adb2e3e8/6b453246-6ae6-4c73-99ea-9f79a5f14ff1"
-					(reference "SB4")
+					(reference "SB803")
 					(unit 1)
 				)
@@
 		(dnp no)
 		(fields_autoplaced yes)
-		(property "Reference" "J18"
+		(property "Reference" "J801"
 			(at 107.95 57.15 0)
 			(effects
@@
 			(project "SACE-HW"
 				(path "/4c1e5ca8-aa0f-4a8e-bffe-6765adb2e3e8/6b453246-6ae6-4c73-99ea-9f79a5f14ff1"
-					(reference "J18")
+					(reference "J801")
 					(unit 1)
 				)
@@
 		(dnp no)
 		(fields_autoplaced yes)
-		(property "Reference" "SB7"
+		(property "Reference" "SB804"
 			(at 175.26 106.68 0)
 			(effects
@@
 			(project "SACE-HW"
 				(path "/4c1e5ca8-aa0f-4a8e-bffe-6765adb2e3e8/6b453246-6ae6-4c73-99ea-9f79a5f14ff1"
-					(reference "SB7")
+					(reference "SB804")
 					(unit 1)
 				)
@@
 		(dnp no)
 		(fields_autoplaced yes)
-		(property "Reference" "SB8"
+		(property "Reference" "SB806"
 			(at 175.26 115.57 0)
 			(effects
@@
 			(project "SACE-HW"
 				(path "/4c1e5ca8-aa0f-4a8e-bffe-6765adb2e3e8/6b453246-6ae6-4c73-99ea-9f79a5f14ff1"
-					(reference "SB8")
+					(reference "SB806")
 					(unit 1)
 				)
@@
 		(on_board yes)
 		(dnp yes)
-		(property "Reference" "R47"
+		(property "Reference" "R804"
 			(at 95.25 115.57 0)
 			(effects
@@
 			(project "SACE-HW"
 				(path "/4c1e5ca8-aa0f-4a8e-bffe-6765adb2e3e8/6b453246-6ae6-4c73-99ea-9f79a5f14ff1"
-					(reference "R47")
+					(reference "R804")
 					(unit 1)
 				)
@@
 		(on_board yes)
 		(dnp no)
-		(property "Reference" "#PWR0136"
+		(property "Reference" "#PWR0803"
 			(at 172.72 74.168 0)
 			(effects
@@
 			(project "SACE-HW"
 				(path "/4c1e5ca8-aa0f-4a8e-bffe-6765adb2e3e8/6b453246-6ae6-4c73-99ea-9f79a5f14ff1"
-					(reference "#PWR0136")
+					(reference "#PWR0803")
 					(unit 1)
 				)
@@
 		(dnp no)
 		(fields_autoplaced yes)
-		(property "Reference" "SB6"
+		(property "Reference" "SB802"
 			(at 175.26 97.79 0)
 			(effects
@@
 			(project "SACE-HW"
 				(path "/4c1e5ca8-aa0f-4a8e-bffe-6765adb2e3e8/6b453246-6ae6-4c73-99ea-9f79a5f14ff1"
-					(reference "SB6")
+					(reference "SB802")
 					(unit 1)
 				)
@@
 		(dnp no)
 		(fields_autoplaced yes)
-		(property "Reference" "R51"
+		(property "Reference" "R802"
 			(at 133.35 66.04 0)
 			(effects
@@
 			(project "SACE-HW"
 				(path "/4c1e5ca8-aa0f-4a8e-bffe-6765adb2e3e8/6b453246-6ae6-4c73-99ea-9f79a5f14ff1"
-					(reference "R51")
+					(reference "R802")
 					(unit 1)
 				)
@@
 		(on_board yes)
 		(dnp no)
-		(property "Reference" "C40"
+		(property "Reference" "C803"
 			(at 147.955 74.93 90)
 			(effects
@@
 			(project "SACE-HW"
 				(path "/4c1e5ca8-aa0f-4a8e-bffe-6765adb2e3e8/6b453246-6ae6-4c73-99ea-9f79a5f14ff1"
-					(reference "C40")
+					(reference "C803")
 					(unit 1)
 				)
@@
 		(dnp no)
 		(fields_autoplaced yes)
-		(property "Reference" "#PWR0134"
+		(property "Reference" "#PWR0801"
 			(at 142.24 58.42 0)
 			(effects
@@
 			(project "SACE-HW"
 				(path "/4c1e5ca8-aa0f-4a8e-bffe-6765adb2e3e8/6b453246-6ae6-4c73-99ea-9f79a5f14ff1"
-					(reference "#PWR0134")
+					(reference "#PWR0801")
 					(unit 1)
 				)
@@
 		(on_board yes)
 		(dnp yes)
-		(property "Reference" "R50"
+		(property "Reference" "R807"
 			(at 95.25 142.24 0)
 			(effects
@@
 			(project "SACE-HW"
 				(path "/4c1e5ca8-aa0f-4a8e-bffe-6765adb2e3e8/6b453246-6ae6-4c73-99ea-9f79a5f14ff1"
-					(reference "R50")
+					(reference "R807")
 					(unit 1)
 				)
@@
 		(on_board yes)
 		(dnp no)
-		(property "Reference" "#PWR0133"
+		(property "Reference" "#PWR0804"
 			(at 129.54 89.408 0)
 			(effects
@@
 			(project "SACE-HW"
 				(path "/4c1e5ca8-aa0f-4a8e-bffe-6765adb2e3e8/6b453246-6ae6-4c73-99ea-9f79a5f14ff1"
-					(reference "#PWR0133")
+					(reference "#PWR0804")
 					(unit 1)
 				)
@@
 		(dnp no)
 		(fields_autoplaced yes)
-		(property "Reference" "#PWR0132"
+		(property "Reference" "#PWR0805"
 			(at 86.36 109.22 0)
 			(effects
@@
 			(project "SACE-HW"
 				(path "/4c1e5ca8-aa0f-4a8e-bffe-6765adb2e3e8/6b453246-6ae6-4c73-99ea-9f79a5f14ff1"
-					(reference "#PWR0132")
+					(reference "#PWR0805")
 					(unit 1)
 				)
@@
 		(on_board yes)
 		(dnp no)
-		(property "Reference" "C41"
+		(property "Reference" "C801"
 			(at 167.64 59.055 90)
 			(effects
@@
 			(project "SACE-HW"
 				(path "/4c1e5ca8-aa0f-4a8e-bffe-6765adb2e3e8/6b453246-6ae6-4c73-99ea-9f79a5f14ff1"
-					(reference "C41")
+					(reference "C801")
 					(unit 1)
 				)
@@
 		(dnp no)
 		(fields_autoplaced yes)
-		(property "Reference" "SB5"
+		(property "Reference" "SB805"
 			(at 156.21 115.57 0)
 			(effects
@@
 			(project "SACE-HW"
 				(path "/4c1e5ca8-aa0f-4a8e-bffe-6765adb2e3e8/6b453246-6ae6-4c73-99ea-9f79a5f14ff1"
-					(reference "SB5")
+					(reference "SB805")
 					(unit 1)
 				)
@@
 		(on_board yes)
 		(dnp yes)
-		(property "Reference" "R49"
+		(property "Reference" "R806"
 			(at 95.25 133.35 0)
 			(effects
@@
 			(project "SACE-HW"
 				(path "/4c1e5ca8-aa0f-4a8e-bffe-6765adb2e3e8/6b453246-6ae6-4c73-99ea-9f79a5f14ff1"
-					(reference "R49")
+					(reference "R806")
 					(unit 1)
 				)
@@
 		(dnp no)
 		(fields_autoplaced yes)
-		(property "Reference" "#PWR0135"
+		(property "Reference" "#PWR0802"
 			(at 172.72 58.42 0)
 			(effects
@@
 			(project "SACE-HW"
 				(path "/4c1e5ca8-aa0f-4a8e-bffe-6765adb2e3e8/6b453246-6ae6-4c73-99ea-9f79a5f14ff1"
-					(reference "#PWR0135")
+					(reference "#PWR0802")
 					(unit 1)
 				)

Commit message: clean up
Parts:
- removed R803, R804, R805, R806, R807: RC0805FR-0747KL, Resistors:R0805, symbol Resistors:RC0805FR-0747KL
- removed SB801, SB802, SB803, SB804, SB805, SB806: Solder_Bridge, Connectors:Solder_bridge_0805, symbol Connectors:Solder_Bridge
Connections:
- net CLK is gone; now on net CARD_SCK: J801.P5 (CLK)
- net CMD is gone; now on net CARD_MOSI: J801.P3 (CMD)
- net DAT0 is gone; now on net CARD_MISO: J801.P7 (DAT0)
- net CARD_CS/DAT3 renamed CARD_CS
- net CARD_DAT1: no longer names the net of J801.P8 (DAT1)
- net CARD_DAT2: no longer names the net of J801.P1 (DAT2)
- no-connect marks 0 -> 2
Other:
- moved on the sheet: C801, C802, C803, J801, R801, R802

Commit message: update
Parts:
- renumbered C801 to C701, C802 to C702, C803 to C703, J801 to J701, R801 to R701, R802 to R702
Changed lines of the file:
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@@
 		(on_board yes)
 		(dnp no)
-		(property "Reference" "C802"
+		(property "Reference" "C702"
 			(at 208.915 54.61 90)
 			(effects
@@
 			(project "SACE-HW"
 				(path "/4c1e5ca8-aa0f-4a8e-bffe-6765adb2e3e8/6b453246-6ae6-4c73-99ea-9f79a5f14ff1"
-					(reference "C802")
+					(reference "C702")
 					(unit 1)
 				)
@@
 		(dnp no)
 		(fields_autoplaced yes)
-		(property "Reference" "R801"
+		(property "Reference" "R701"
 			(at 166.37 58.42 90)
 			(effects
@@
 			(project "SACE-HW"
 				(path "/4c1e5ca8-aa0f-4a8e-bffe-6765adb2e3e8/6b453246-6ae6-4c73-99ea-9f79a5f14ff1"
-					(reference "R801")
+					(reference "R701")
 					(unit 1)
 				)
@@
 		(dnp no)
 		(fields_autoplaced yes)
-		(property "Reference" "J801"
+		(property "Reference" "J701"
 			(at 129.54 52.07 0)
 			(effects
@@
 			(project "SACE-HW"
 				(path "/4c1e5ca8-aa0f-4a8e-bffe-6765adb2e3e8/6b453246-6ae6-4c73-99ea-9f79a5f14ff1"
-					(reference "J801")
+					(reference "J701")
 					(unit 1)
 				)
@@
 		(on_board yes)
 		(dnp no)
-		(property "Reference" "#PWR0803"
+		(property "Reference" "#PWR0703"
 			(at 194.31 69.088 0)
 			(effects
@@
 			(project "SACE-HW"
 				(path "/4c1e5ca8-aa0f-4a8e-bffe-6765adb2e3e8/6b453246-6ae6-4c73-99ea-9f79a5f14ff1"
-					(reference "#PWR0803")
+					(reference "#PWR0703")
 					(unit 1)
 				)
@@
 		(dnp no)
 		(fields_autoplaced yes)
-		(property "Reference" "R802"
+		(property "Reference" "R702"
 			(at 154.94 60.96 0)
 			(effects
@@
 			(project "SACE-HW"
 				(path "/4c1e5ca8-aa0f-4a8e-bffe-6765adb2e3e8/6b453246-6ae6-4c73-99ea-9f79a5f14ff1"
-					(reference "R802")
+					(reference "R702")
 					(unit 1)
 				)
@@
 		(on_board yes)
 		(dnp no)
-		(property "Reference" "C803"
+		(property "Reference" "C703"
 			(at 169.545 69.85 90)
 			(effects
@@
 			(project "SACE-HW"
 				(path "/4c1e5ca8-aa0f-4a8e-bffe-6765adb2e3e8/6b453246-6ae6-4c73-99ea-9f79a5f14ff1"
-					(reference "C803")
+					(reference "C703")
 					(unit 1)
 				)
@@
 		(dnp no)
 		(fields_autoplaced yes)
-		(property "Reference" "#PWR0801"
+		(property "Reference" "#PWR0701"
 			(at 163.83 53.34 0)
 			(effects
@@
 			(project "SACE-HW"
 				(path "/4c1e5ca8-aa0f-4a8e-bffe-6765adb2e3e8/6b453246-6ae6-4c73-99ea-9f79a5f14ff1"
-					(reference "#PWR0801")
+					(reference "#PWR0701")
 					(unit 1)
 				)
@@
 		(on_board yes)
 		(dnp no)
-		(property "Reference" "#PWR0804"
+		(property "Reference" "#PWR0704"
 			(at 151.13 84.328 0)
 			(effects
@@
 			(project "SACE-HW"
 				(path "/4c1e5ca8-aa0f-4a8e-bffe-6765adb2e3e8/6b453246-6ae6-4c73-99ea-9f79a5f14ff1"
-					(reference "#PWR0804")
+					(reference "#PWR0704")
 					(unit 1)
 				)
@@
 		(on_board yes)
 		(dnp no)
-		(property "Reference" "C801"
+		(property "Reference" "C701"
 			(at 189.23 53.975 90)
 			(effects
@@
 		)
 		(property "Capacitance (Farad)" "1µF"
-			(at 189.23 57.1499 90)
-			(effects
-				(font
-					(size 1.27 1.27)
-				)
-				(justify right)
+			(at 188.468 55.88 0)
+			(effects
+				(font
+					(size 1.27 1.27)
+				)
 			)
 		)
@@
 			(project "SACE-HW"
 				(path "/4c1e5ca8-aa0f-4a8e-bffe-6765adb2e3e8/6b453246-6ae6-4c73-99ea-9f79a5f14ff1"
-					(reference "C801")
+					(reference "C701")
 					(unit 1)
 				)
@@
 		(dnp no)
 		(fields_autoplaced yes)
-		(property "Reference" "#PWR0802"
+		(property "Reference" "#PWR0702"
 			(at 194.31 53.34 0)
 			(effects
@@
 			(project "SACE-HW"
 				(path "/4c1e5ca8-aa0f-4a8e-bffe-6765adb2e3e8/6b453246-6ae6-4c73-99ea-9f79a5f14ff1"
-					(reference "#PWR0802")
+					(reference "#PWR0702")
 					(unit 1)
 				)
