File: carte_controle/MCU.kicad_sch (KiCad schematic)
At the start: 11 parts, among them SW301 PTS645SM43SMTR92, U301 ESP32-DEVKITC-32D

Commit message: parts placement finished
Parts:
- added R306: RC0805JR-0710KL, Resistors:R0805, symbol Resistors:RC0805JR-0710KL
Connections:
- net VDD: now also R306.1; no longer U301.J2-2 (EN)
- new net: R306.2, U301.J2-2 (EN)
- no-connect marks 2 -> 3
Changed lines of the file:
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@@
-	)
-	(junction
-		(at 109.22 59.69)
-		(diameter 0)
-		(color 0 0 0 0)
 	)
 	(junction
@@
 		(color 0 0 0 0)
 	)
+	(junction
+		(at 91.44 59.69)
+		(diameter 0)
+		(color 0 0 0 0)
+	)
 	(no_connect
 		(at 236.22 83.82)
@@
 		(at 238.76 93.98)
 	)
+	(no_connect
+		(at 114.3 105.41)
+	)
 	(wire
 		(pts
@@
 	(wire
 		(pts
-			(xy 109.22 59.69) (xy 114.3 59.69)
+			(xy 91.44 59.69) (xy 114.3 59.69)
 		)
 		(stroke
@@
 	(wire
 		(pts
-			(xy 109.22 58.42) (xy 109.22 59.69)
-		)
-		(stroke
-			(width 0)
-			(type default)
-		)
-	)
-	(wire
-		(pts
-			(xy 114.3 62.23) (xy 109.22 62.23)
+			(xy 91.44 50.8) (xy 91.44 59.69)
+		)
+		(stroke
+			(width 0)
+			(type default)
+		)
+	)
+	(wire
+		(pts
+			(xy 102.87 62.23) (xy 114.3 62.23)
 		)
 		(stroke
@@
 	(wire
 		(pts
-			(xy 109.22 62.23) (xy 109.22 59.69)
-		)
-		(stroke
-			(width 0)
-			(type default)
-		)
-	)
-	(wire
-		(pts
 			(xy 113.03 67.31) (xy 114.3 67.31)
 		)
@@
 	(wire
 		(pts
+			(xy 91.44 62.23) (xy 91.44 59.69)
+		)
+		(stroke
+			(width 0)
+			(type default)
+		)
+	)
+	(wire
+		(pts
 			(xy 238.76 66.04) (xy 238.76 68.58)
 		)
@@
 		(pts
 			(xy 106.68 163.83) (xy 162.56 163.83)
+		)
+		(stroke
+			(width 0)
+			(type default)
+		)
+	)
+	(wire
+		(pts
+			(xy 92.71 62.23) (xy 91.44 62.23)
 		)
 		(stroke
@@
 	(symbol
 		(lib_id "Power_Port:VDD")
-		(at 109.22 58.42 0)
+		(at 91.44 50.8 0)
 		(unit 1)
 		(exclude_from_sim no)
@@
 		(fields_autoplaced yes)
 		(property "Reference" "#PWR0301"
-			(at 109.22 62.23 0)
+			(at 91.44 54.61 0)
 			(effects
 				(font
@@
 		)
 		(property "Value" "VDD"
-			(at 109.22 53.34 0)
+			(at 91.44 45.72 0)
 			(effects
 				(font
@@
 		)
 		(property "Footprint" ""
-			(at 109.22 58.42 0)
+			(at 91.44 50.8 0)
 			(effects
 				(font
@@
 		)
 		(property "Datasheet" ""
-			(at 109.22 62.23 0)
+			(at 91.44 54.61 0)
 			(effects
 				(font
@@
 		)
 		(property "Description" ""
-			(at 109.22 58.42 0)
+			(at 91.44 50.8 0)
 			(effects
 				(font
@@
 					(unit 1)
 				)
+			)
+		)
+	)
+	(symbol
+		(lib_id "Resistors:RC0805JR-0710KL")
+		(at 97.79 62.23 0)
+		(mirror x)
+		(unit 1)
+		(exclude_from_sim no)
+		(in_bom yes)
+		(on_board yes)
+		(dnp no)
+		(property "Reference" "R306"
+			(at 97.79 67.31 0)
+			(effects
+				(font
+					(size 1.524 1.524)
+				)
+			)
+		)
+		(property "Value" "RC0805JR-0710KL"
+			(at 97.79 54.61 0)
+			(effects
+				(font
+					(size 1.27 1.27)
+				)
+				(hide yes)
+			)
+		)
+		(property "Footprint" "Resistors:R0805"
+			(at 97.79 39.37 0)
+			(effects
+				(font
+					(size 0.762 0.762)
+				)
+				(hide yes)
+			)
+		)
+		(property "Datasheet" "http://www.yageo.com/documents/recent/PYu-RC_Group_51_RoHS_L_7.pdf"
+			(at 97.79 38.1 0)
+			(effects
+				(font
+					(size 0.762 0.762)
+				)
+				(hide yes)
+			)
+		)
+		(property "Description" "RES SMD 10K OHM 5% 1/8W 0805"
+			(at 97.79 41.91 0)
+			(effects
+				(font
+					(size 1.524 1.524)
+				)
+				(hide yes)
+			)
+		)
+		(property "Supplier" "Digikey"
+			(at 97.79 52.07 0)
+			(effects
+				(font
+					(size 1.524 1.524)
+				)
+				(hide yes)
+			)
+		)
+		(property "Supplier Part Number" "311-10KARCT-ND"
+			(at 97.79 49.53 0)
+			(effects
+				(font
+					(size 1.524 1.524)
+				)
+				(hide yes)
+			)
+		)
+		(property "Manufacturer" "Yageo"
+			(at 97.79 46.99 0)
+			(effects
+				(font
+					(size 1.524 1.524)
+				)
+				(hide yes)
+			)
+		)
+		(property "Manufacturer Part Number" "RC0805JR-0710KL"
+			(at 97.79 44.45 0)
+			(effects
+				(font
+					(size 1.524 1.524)
+				)
+				(hide yes)
+			)
+		)
+		(property "Resistance (Ohms)" "10k"
+			(at 97.79 64.77 0)
+			(effects
+				(font
+					(size 1.27 1.27)
+				)
+			)
+		)
+		(property "Tolerance (%)" "±5%"
+			(at 108.204 60.198 0)
+			(effects
+				(font
+					(size 1.27 1.27)
+				)
+				(hide yes)
+			)
+		)
+		(property "Puissance (Watts)" "1/8W"
+			(at 97.79 58.674 0)
+			(effects
+				(font
+					(size 1.27 1.27)
+				)
+				(hide yes)
+			)
+		)
+		(pin "2"
+		)
+		(pin "1"
+		)
+		(instances
+			(project "SACE-HW"
+				(path "/4c1e5ca8-aa0f-4a8e-bffe-6765adb2e3e8/558e191e-4d57-467a-8f3d-07afb9cf3132"
+					(reference "R306")
+					(unit 1)
+				)
