File: carte_controle/SACE-HW.kicad_sch (KiCad schematic)
At the start: 5 parts, among them J101 2350514-8

Commit message: parts placement finished
Parts:
- removed J101: 2350514-8, Connectors:CONN8_2350514-8_TEC, symbol Connectors:2350514-8
Connections:
- no-connect marks 9 -> 8
Other:
- sheet 5V_OUTPUT ports: added NO_1, NO_2; removed none
- sheet I2C ports: added HV_EN, LDAC_A, LDAC_B, SCL, SDA; removed SCL_5V, SDA_5V
