File: carte_controle/HV.kicad_sch (KiCad schematic)
At the start: 29 parts, among them J401 1935161, J402 1935161, J403 RF1-01K-D-00-50-BK-HDW, J404 RF1-01K-D-00-50-BK-HDW, Q401 MCB90N12A-TP, U401 LTV-816S, U402 ADC124S021CIMM, U403 TMCS1101A3UQDT, U404 ISO7341CQDWQ1, U405 MCP6L04T-E/SL

Commit message: gerber + commande JLC
Connections:
- net HV: now also F401.2; no longer J402.2, R405.2
- net e-: now also Q401.2 (D); no longer F401.2
- net e+: now reaches F401.1
- net e+: now also J402.2, R405.2; no longer Q401.2 (D)
Other:
- moved on the sheet: F401, J402
Changed lines of the file:
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@@
 	)
 	(junction
-		(at 114.3 26.67)
-		(diameter 0)
-		(color 0 0 0 0)
-	)
-	(junction
 		(at 53.34 140.97)
 		(diameter 0)
@@
 	)
 	(junction
-		(at 114.3 29.21)
-		(diameter 0)
-		(color 0 0 0 0)
-	)
-	(junction
 		(at 31.75 76.2)
 		(diameter 0)
@@
 	(wire
 		(pts
-			(xy 114.3 26.67) (xy 120.65 26.67)
-		)
-		(stroke
-			(width 0)
-			(type default)
-		)
-	)
-	(wire
-		(pts
 			(xy 33.02 76.2) (xy 31.75 76.2)
 		)
@@
 	(wire
 		(pts
-			(xy 114.3 29.21) (xy 120.65 29.21)
-		)
-		(stroke
-			(width 0)
-			(type default)
-		)
-	)
-	(wire
-		(pts
 			(xy 81.28 143.51) (xy 80.01 143.51)
 		)
@@
 	(wire
 		(pts
-			(xy 114.3 21.59) (xy 114.3 26.67)
-		)
-		(stroke
-			(width 0)
-			(type default)
-		)
-	)
-	(wire
-		(pts
 			(xy 134.62 73.66) (xy 137.16 73.66)
 		)
@@
 	(wire
 		(pts
+			(xy 107.95 38.1) (xy 114.3 38.1)
+		)
+		(stroke
+			(width 0)
+			(type default)
+		)
+	)
+	(wire
+		(pts
 			(xy 81.28 113.03) (xy 80.01 113.03)
 		)
@@
 	(wire
 		(pts
-			(xy 111.76 29.21) (xy 114.3 29.21)
+			(xy 114.3 38.1) (xy 114.3 40.64)
 		)
 		(stroke
@@
 	(wire
 		(pts
-			(xy 114.3 26.67) (xy 111.76 26.67)
+			(xy 107.95 35.56) (xy 114.3 35.56)
 		)
 		(stroke
@@
 	(wire
 		(pts
+			(xy 114.3 31.75) (xy 114.3 35.56)
+		)
+		(stroke
+			(width 0)
+			(type default)
+		)
+	)
+	(wire
+		(pts
 			(xy 31.75 76.2) (xy 31.75 77.47)
 		)
@@
 	(wire
 		(pts
-			(xy 114.3 39.37) (xy 114.3 40.64)
-		)
-		(stroke
-			(width 0)
-			(type default)
-		)
-	)
-	(wire
-		(pts
 			(xy 134.62 68.58) (xy 148.59 68.58)
 		)
@@
 	)
 	(label "e-"
-		(at 120.65 29.21 180)
+		(at 114.3 38.1 180)
 		(fields_autoplaced yes)
 		(effects
@@
 	)
 	(label "e+"
-		(at 120.65 26.67 180)
+		(at 114.3 35.56 180)
 		(fields_autoplaced yes)
 		(effects
@@
 	(symbol
 		(lib_id "Connectors:1935161")
-		(at 109.22 29.21 0)
+		(at 105.41 38.1 0)
 		(unit 1)
 		(exclude_from_sim no)
@@
 		(fields_autoplaced yes)
 		(property "Reference" "J402"
-			(at 107.315 22.86 0)
+			(at 103.505 31.75 0)
 			(effects
 				(font
@@
 		)
 		(property "Value" "1935161"
-			(at 109.22 37.338 0)
+			(at 105.41 46.228 0)
 			(effects
 				(font
@@
 		)
 		(property "Footprint" "Connectors:1935161"
-			(at 109.22 52.324 0)
+			(at 105.41 61.214 0)
 			(effects
 				(font
@@
 		)
 		(property "Datasheet" "https://media.digikey.com/pdf/Data%20Sheets/Phoenix%20Contact%20PDFs/1935161.pdf"
-			(at 109.22 53.594 0)
+			(at 105.41 62.484 0)
 			(effects
 				(font
@@
 		)
 		(property "Description" "TERM BLOCK PCB 2POS 5.0MM GREEN"
-			(at 109.22 49.784 0)
+			(at 105.41 58.674 0)
 			(effects
 				(font
@@
 		)
 		(property "Supplier" "Digikey"
-			(at 109.22 42.164 0)
+			(at 105.41 51.054 0)
 			(effects
 				(font
@@
 		)
 		(property "Supplier Part Number" "277-1667-ND"
-			(at 109.22 39.624 0)
+			(at 105.41 48.514 0)
 			(effects
 				(font
@@
 		)
 		(property "Manufacturer" "Phoenix Contact"
-			(at 109.22 44.704 0)
+			(at 105.41 53.594 0)
 			(effects
 				(font
@@
 		)
 		(property "Manufacturer Part Number" "1935161"
-			(at 109.22 47.244 0)
+			(at 105.41 56.134 0)
 			(effects
 				(font
@@
 	(symbol
 		(lib_id "Fuses:0698Q6300-01")
-		(at 114.3 34.29 90)
+		(at 114.3 26.67 90)
 		(unit 1)
 		(exclude_from_sim no)
@@
 		(fields_autoplaced yes)
 		(property "Reference" "F401"
-			(at 116.84 33.0199 90)
+			(at 116.84 25.3999 90)
 			(effects
 				(font
@@
 		)
 		(property "Value" "0698Q6300-01"
-			(at 121.92 34.29 0)
+			(at 121.92 26.67 0)
 			(effects
 				(font
@@
 		)
 		(property "Footprint" "Fuses:TE5_395"
-			(at 137.16 34.29 0)
+			(at 137.16 26.67 0)
 			(effects
 				(font
@@
 		)
 		(property "Datasheet" "https://belfuse.com/resources/CircuitProtection/datasheets/0698Q%20Mar2016.pdf"
-			(at 138.43 34.29 0)
+			(at 138.43 26.67 0)
 			(effects
 				(font
@@
 		)
 		(property "Description" "FUSE BOARD MNT 6.3A 350VAC 140VDC"
-			(at 114.3 34.29 0)
+			(at 114.3 26.67 0)
 			(effects
 				(font
@@
 		)
 		(property "Supplier" "Digikey"
-			(at 124.46 34.29 0)
+			(at 124.46 26.67 0)
 			(effects
 				(font
@@
 		)
 		(property "Supplier Part Number" "507-1848-ND"
-			(at 127 34.29 0)
+			(at 127 26.67 0)
 			(effects
 				(font
@@
 		)
 		(property "Manufacturer" "Bel Fuse Inc."
-			(at 129.54 34.29 0)
+			(at 129.54 26.67 0)
 			(effects
 				(font
@@
 		)
 		(property "Manufacturer Part Number" "0698Q6300-01"
-			(at 132.08 34.29 0)
+			(at 132.08 26.67 0)
 			(effects
 				(font
@@
 		)
 		(property "Description_1" "FUSE BOARD MNT 6.3A 350VAC 140VDC"
-			(at 134.62 34.29 0)
+			(at 134.62 26.67 0)
 			(effects
 				(font
@@
 		)
 		(property "Current Rating (A)" "6.3A"
-			(at 116.84 35.5599 90)
+			(at 116.84 27.9399 90)
 			(effects
 				(font
@@
 		)
 		(property "Voltage Rating - DC" "140VDC"
-			(at 119.38 39.37 0)
+			(at 119.38 31.75 0)
 			(effects
 				(font
@@
 		)
 		(property "Voltage Rating - AC" "350VAC"
-			(at 119.38 29.21 0)
+			(at 119.38 21.59 0)
 			(effects
 				(font
