File: carte_controle/SACE-HW.kicad_pcb (KiCad board)
At the start: 2 copper layers, 100 x 160 mm, 133 parts, among them IC201 1769205241, J101 2350514-8, J201 Header_Male_Pin_2.54mm_1X2_,_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, J202 1935161, J203 2350514-8, J401 1935161, J402 1935161, J403 RF1-01K-D-00-50-BK-HDW, J404 RF1-01K-D-00-50-BK-HDW, J501 2350514-8, J502 XH-4A connector, J503 XH-4A connector, J504 2350514-8, J505 2350514-8, J601 2350514-8, J701 MEM2075-00-140-01-A, J801 2350514-4, J802 2350514-8, Q401 MCB90N12A-TP, Q801 PMV20XNER, Q802 PMV20XNER, Q803 PMV20XNER, Q804 PMV20XNER, Q805 PMV20XNER, Q806 PMV20XNER, SW301 PTS645SM43SMTR92, U201 AZ1117IH-3.3TRG1, U202 OKI-78SR-5_1.5-W36H-C, U203 AZ1117IH-3.3TRG1, U301 ESP32-DEVKITC-32D, U401 LTV-816S, U402 ADC124S021CIMM, U403 TMCS1101A3UQDT, U404 ISO7341CQDWQ1, U405 MCP6L04T-E/SL, U501 MCP4728T-E_UN, U502 TLV9302IDR, U503 TLA2528IRTER, U504 TCA9617BDGKR, U601 74LVC4245APW_118

Commit message: parts placement finished
Parts:
- removed J101: 2350514-8, Connectors:CONN8_2350514-8_TEC
- added J602: 2350514-4, Connectors:CONN4_1155650000_TEC, F.Cu at (77.8, 76.3)
- added R306: RC0805JR-0710KL, Resistors:R0805, F.Cu at (125.5, 137.9)
- added R514: RC0805JR-07100KL, Resistors:R0805, F.Cu at (88.4, 117.1)
- added R515: RC0805JR-072K2L, Resistors:R0805, F.Cu at (125.1, 89.2)
- added R516: RC0805JR-072K2L, Resistors:R0805, F.Cu at (89.7, 61.7)
- added R517: RC0805JR-07100KL, Resistors:R0805, F.Cu at (86.6, 53.8)
- added R518: RC0805JR-074K7L, Resistors:R0805, F.Cu at (91.2, 55.8)
- added R519: RC0805JR-074K7L, Resistors:R0805, F.Cu at (93.5, 55.8)
- added R520: RC0805JR-072K2L, Resistors:R0805, F.Cu at (130.5, 89.2)
- added U505: SI8602AC-B-IS, IC:SOIC-8, F.Cu at (116.0, 81.0)
- added U506: MCP4728T-E_UN, IC:SOP50P490X110-10N, F.Cu at (85.0, 60.5)
- added U507: LTV-816S, IC:4-SMD, F.Cu at (123.8, 81.0)
- added U508: LTV-816S, IC:4-SMD, F.Cu at (129.2, 81.0)
- added U602: LTV-816S, IC:4-SMD, F.Cu at (84.5, 95.0)
- added U603: LTV-816S, IC:4-SMD, F.Cu at (91.6, 95.0)
- J504: value 2350514-8 -> 2350514-4; footprint Connectors:CONN8_2350514-8_TEC -> Connectors:CONN4_1155650000_TEC
- moved C401 112.9 mm to (107.1, 67.4), turned to 90 degrees
- moved C402 108.9 mm to (109.5, 67.4), turned to 90 degrees
- moved J504 101.0 mm to (77.9, 58.1)
- moved R403 100.7 mm to (135.8, 91.1), turned to 90 degrees
- moved C403 95.3 mm to (147.0, 71.1), turned to 180 degrees
- moved J203 92.0 mm to (160.9, 117.5), turned to -90 degrees
- moved C404 89.9 mm to (147.0, 68.8), turned to 180 degrees
- moved R401 82.7 mm to (144.7, 62.3), turned to -90 degrees
- moved U405 79.9 mm to (148.8, 55.3)
- moved R411 75.9 mm to (156.8, 59.0), turned to 180 degrees
- moved R407 74.5 mm to (156.9, 51.7), turned to 180 degrees
- moved R410 74.4 mm to (142.9, 58.5), turned to 180 degrees
- moved C405 74.1 mm to (140.9, 53.9)
- moved C406 72.9 mm to (140.9, 55.9)
- moved R406 72.7 mm to (156.8, 54.0), turned to 180 degrees
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Connections:
- J502 pad 2: /IO21 -> /I2C/SDA_5V
- J502 pad 3: /IO22 -> /I2C/SCL_5V
- J503 pad 2: /IO21 -> /I2C/SDA_5V
- J503 pad 3: /IO22 -> /I2C/SCL_5V
- J504 pad 1: /I2C/GPIO0 -> Net-(U506-VOUTA)
- J504 pad 2: GNDB -> Net-(U506-VOUTB)
- J504 pad 3: /I2C/GPIO1 -> Net-(U508-C)
- J504 pad 4: GNDB -> Net-(U508-E)
- J505 pad 1: /I2C/GPIO4 -> Net-(U503-AIN0/GPIO0)
- J505 pad 2: GNDB -> Net-(U503-AIN1/GPIO1)
- J505 pad 3: /I2C/GPIO5 -> Net-(U503-AIN2/GPIO2)
- J505 pad 4: GNDB -> Net-(U503-AIN3/GPIO3)
- J505 pad 5: /I2C/GPIO6 -> Net-(U503-AIN4/GPIO4)
- J505 pad 6: GNDB -> Net-(U503-AIN5/GPIO5)
- J505 pad 7: /I2C/GPIO7 -> Net-(U503-AIN6/GPIO6)
- J505 pad 8: GNDB -> Net-(U503-AIN7/GPIO7)
- R501 pad 1: /IO22 -> /I2C/SCL_5V
- R502 pad 1: /IO21 -> /I2C/SDA_5V
- R503 pad 1: /I2C/SCL -> /IO22
- R504 pad 1: /I2C/SDA -> /IO21
- U301 pad J2-11: /MCU/IO27 -> /IO27
- U301 pad J2-2: VDD -> Net-(U301-EN)
- U501 pad 2: /IO22 -> /I2C/SCL_5V
- U501 pad 3: /IO21 -> /I2C/SDA_5V
- U501 pad 4: unconnected-(U501-*LDAC-Pad4) -> /IO33
- U501 pad 5: unconnected-(U501-RDY/*BSY-Pad5) -> Net-(U501-RDY/*BSY)
- U503 pad 1: /I2C/GPIO2 -> Net-(U503-AIN2/GPIO2)
- U503 pad 13: /IO22 -> /I2C/SCL_5V
- U503 pad 14: /IO21 -> /I2C/SDA_5V
- U503 pad 15: /I2C/GPIO0 -> Net-(U503-AIN0/GPIO0)
- U503 pad 16: /I2C/GPIO1 -> Net-(U503-AIN1/GPIO1)
- U503 pad 2: /I2C/GPIO3 -> Net-(U503-AIN3/GPIO3)
- U503 pad 3: /I2C/GPIO4 -> Net-(U503-AIN4/GPIO4)
- U503 pad 4: /I2C/GPIO5 -> Net-(U503-AIN5/GPIO5)
- U503 pad 5: /I2C/GPIO6 -> Net-(U503-AIN6/GPIO6)
- U503 pad 6: /I2C/GPIO7 -> Net-(U503-AIN7/GPIO7)
- U504 pad 2: /I2C/SCL -> /IO22
- U504 pad 3: /I2C/SDA -> /IO21
- U504 pad 6: /IO21 -> /I2C/SDA_5V
- U504 pad 7: /IO22 -> /I2C/SCL_5V

Commit message: gerber + commande JLC
Parts:
- moved U603 14.2 mm to (89.0, 81.0)
- moved U602 14.1 mm to (83.0, 81.0)
- moved IC201 11.0 mm to (114.0, 81.8)
- moved F201 10.9 mm to (104.3, 75.4), turned to 90 degrees
- moved J504 10.7 mm to (78.0, 47.4)
- moved J602 10.4 mm to (78.0, 65.9)
- moved U505 8.42 mm to (124.4, 80.6)
- moved U201 8.00 mm to (97.4, 75.1)
- moved R401 7.42 mm to (151.9, 64.1), turned to 180 degrees
- moved C201 7.34 mm to (91.6, 71.6)
- moved C202 7.34 mm to (91.6, 69.3)
- moved U506 7.21 mm to (85.4, 53.3)
- moved R515 7.20 mm to (132.3, 89.2)
- moved U508 7.20 mm to (136.4, 81.0)
- moved U507 7.20 mm to (131.0, 81.0)
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Connections:
- F401 pad 1: Net-(Q401-D) -> /HV/e+
- F401 pad 2: /HV/e- -> HV
- J402 pad 2: HV -> /HV/e+
- Q401 pad 2: Net-(Q401-D) -> /HV/e-
- R405 pad 2: HV -> /HV/e+
Routing:
- net 5VB: track 0.00 -> 280.6 mm, vias 0 -> 4
- net 12VB: track 0.00 -> 253.7 mm, vias 0 -> 1
- net VDD: track 0.00 -> 194.0 mm, vias 0 -> 2
- net 5VA: track 0.00 -> 179.5 mm, vias 0 -> 1
- net /IO12: track 0.00 -> 147.5 mm, vias 0 -> 2
- net /IO13: track 0.00 -> 138.2 mm, vias 0 -> 2
- net /I2C/SDA_5V: track 0.00 -> 137.0 mm, vias 0 -> 3
- net /IO14: track 0.00 -> 135.0 mm, vias 0 -> 3
- net /IO27: track 0.00 -> 129.3 mm, vias 0 -> 1
- net /I2C/SCL_5V: track 0.00 -> 129.1 mm, vias 0 -> 4
- net 3.3VB: track 0.00 -> 110.4 mm, vias 0 -> 1
- net /IO15: track 0.00 -> 103.5 mm
- net /IO0: track 0.00 -> 99.6 mm
- net /IO1: track 0.00 -> 99.0 mm, vias 0 -> 1
- net /HV/V_amp: track 0.00 -> 98.6 mm, vias 0 -> 2
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- added copper zone on B.Cu, net GNDA
- added copper zone on F.Cu, net GNDA
- added copper zone on B.Cu, net GNDB
- added copper zone on F.Cu, net GNDB
Other:
- board text added: "12VB"
- board text added: "3.3VA"
- board text added: "3.3VB"
- board text added: "5VA"
- board text added: "5VB"
- board text added: "HV SIDE"
- board text added: "SACE HW V1 - 2024 Gérémy Sauvageau"
- board text removed: "3.3V (A)"
- board text removed: "5V (A)"
