File: interface_piezzos/piezzo/piezzo.kicad_pcb (KiCad board)
At the start: 2 copper layers, 34.4 x 21.7 mm, 16 parts, among them J101 2350514-4, U101 TLV9302IDR

Commit message: gerber + commande JLC
Parts:
- added Z1: MMSZ5231B, Diodes:SOD-123FL, F.Cu at (150.1, 80.1)
- moved VR101 1.15 mm to (150.4, 73.8)
- moved C102 0.85 mm to (157.9, 82.0)
- moved C103 0.85 mm to (157.9, 79.8)
Routing:
- net Net-(TP101-TP): track 46.7 -> 49.8 mm
- net 5V: track 18.9 -> 20.4 mm
- net Net-(C101-Pad2): track 14.9 -> 16.1 mm
Other:
- board text added: "TRIG ADJUST"
