File: interface_piezzos/piezzo.kicad_sch (KiCad schematic)
At the start: 17 parts, among them J101 2350514-4, U101 TLV9302IDR

Commit message: un peu d'ordre la dedans
Other:
- company: (none) -> Gérémy Sauvageau
- title: (none) -> PIEZZO
- moved on the sheet: C102, C103
Changed lines of the file:
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@@
 	(generator_version "8.0")
 	(paper "A4")
+	(title_block
+		(title "PIEZZO")
+		(date "2024-07-24")
+		(company "Gérémy Sauvageau")
+	)
 	(junction
 		(at 101.6 60.96)
@@
 	)
 	(junction
-		(at 182.88 66.04)
+		(at 166.37 64.77)
 		(diameter 0)
 		(color 0 0 0 0)
@@
 	)
 	(junction
-		(at 182.88 50.8)
+		(at 166.37 49.53)
 		(diameter 0)
 		(color 0 0 0 0)
@@
 	(wire
 		(pts
-			(xy 186.69 66.04) (xy 186.69 63.5)
-		)
-		(stroke
-			(width 0)
-			(type default)
-		)
-	)
-	(wire
-		(pts
-			(xy 186.69 50.8) (xy 182.88 50.8)
+			(xy 170.18 64.77) (xy 170.18 62.23)
+		)
+		(stroke
+			(width 0)
+			(type default)
+		)
+	)
+	(wire
+		(pts
+			(xy 170.18 49.53) (xy 166.37 49.53)
 		)
 		(stroke
@@
 	(wire
 		(pts
-			(xy 177.8 66.04) (xy 182.88 66.04)
+			(xy 161.29 64.77) (xy 166.37 64.77)
 		)
 		(stroke
@@
 	(wire
 		(pts
-			(xy 186.69 55.88) (xy 186.69 50.8)
-		)
-		(stroke
-			(width 0)
-			(type default)
-		)
-	)
-	(wire
-		(pts
-			(xy 177.8 55.88) (xy 177.8 50.8)
+			(xy 170.18 54.61) (xy 170.18 49.53)
+		)
+		(stroke
+			(width 0)
+			(type default)
+		)
+	)
+	(wire
+		(pts
+			(xy 161.29 54.61) (xy 161.29 49.53)
 		)
 		(stroke
@@
 	(wire
 		(pts
-			(xy 177.8 63.5) (xy 177.8 66.04)
+			(xy 161.29 62.23) (xy 161.29 64.77)
 		)
 		(stroke
@@
 	(wire
 		(pts
-			(xy 182.88 66.04) (xy 186.69 66.04)
+			(xy 166.37 64.77) (xy 170.18 64.77)
 		)
 		(stroke
@@
 	(wire
 		(pts
-			(xy 177.8 50.8) (xy 182.88 50.8)
+			(xy 161.29 49.53) (xy 166.37 49.53)
 		)
 		(stroke
@@
 	(symbol
 		(lib_id "Power_Port:DGND")
-		(at 182.88 68.58 0)
+		(at 166.37 67.31 0)
 		(unit 1)
 		(exclude_from_sim no)
@@
 		(dnp no)
 		(property "Reference" "#PWR0108"
-			(at 182.88 72.898 0)
+			(at 166.37 71.628 0)
 			(effects
 				(font
@@
 		)
 		(property "Value" "DGND"
-			(at 186.182 71.374 0)
+			(at 169.672 70.104 0)
 			(effects
 				(font
@@
 		)
 		(property "Footprint" ""
-			(at 182.88 66.04 0)
+			(at 166.37 64.77 0)
 			(effects
 				(font
@@
 		)
 		(property "Datasheet" ""
-			(at 182.372 70.866 0)
+			(at 165.862 69.596 0)
 			(effects
 				(font
@@
 		)
 		(property "Description" ""
-			(at 182.88 68.58 0)
+			(at 166.37 67.31 0)
 			(effects
 				(font
@@
 	(symbol
 		(lib_id "Power_Port:5V")
-		(at 182.88 50.8 0)
+		(at 166.37 49.53 0)
 		(unit 1)
 		(exclude_from_sim no)
@@
 		(fields_autoplaced yes)
 		(property "Reference" "#PWR0107"
-			(at 182.88 54.61 0)
+			(at 166.37 53.34 0)
 			(effects
 				(font
@@
 		)
 		(property "Value" "5V"
-			(at 182.88 45.72 0)
+			(at 166.37 44.45 0)
 			(effects
 				(font
@@
 		)
 		(property "Footprint" ""
-			(at 182.88 50.8 0)
+			(at 166.37 49.53 0)
 			(effects
 				(font
@@
 		)
 		(property "Datasheet" ""
-			(at 182.88 50.8 0)
+			(at 166.37 49.53 0)
 			(effects
 				(font
@@
 		)
 		(property "Description" ""
-			(at 182.88 50.8 0)
+			(at 166.37 49.53 0)
 			(effects
 				(font
@@
 	(symbol
 		(lib_id "Capacitors:885012107015")
-		(at 177.8 58.42 90)
+		(at 161.29 57.15 90)
 		(unit 1)
 		(exclude_from_sim no)
@@
 		(fields_autoplaced yes)
 		(property "Reference" "C103"
-			(at 181.61 57.7849 90)
+			(at 165.1 56.5149 90)
 			(effects
 				(font
@@
 		)
 		(property "Value" "885012107015"
-			(at 186.69 59.69 0)
+			(at 170.18 58.42 0)
 			(effects
 				(font
@@
 		)
 		(property "Footprint" "Capacitors:C0805"
-			(at 201.93 59.69 0)
+			(at 185.42 58.42 0)
 			(effects
 				(font
@@
 		)
 		(property "Datasheet" "D"
-			(at 204.47 59.69 0)
+			(at 187.96 58.42 0)
 			(effects
 				(font
@@
 		)
 		(property "Description" "CAP CER 1UF 25V X5R 0805"
-			(at 199.39 59.69 0)
+			(at 182.88 58.42 0)
 			(effects
 				(font
@@
 		)
 		(property "Supplier" "Digikey"
-			(at 189.23 59.69 0)
+			(at 172.72 58.42 0)
 			(effects
 				(font
@@
 		)
 		(property "Supplier Part Number" "732-7625-1-ND"
-			(at 191.77 59.69 0)
+			(at 175.26 58.42 0)
 			(effects
 				(font
@@
 		)
 		(property "Manufacturer" "Wurth Electronics Inc."
-			(at 194.31 59.69 0)
+			(at 177.8 58.42 0)
 			(effects
 				(font
@@
 		)
 		(property "Manufacturer Part Number" "885012107015"
-			(at 196.85 59.69 0)
+			(at 180.34 58.42 0)
 			(effects
 				(font
@@
 		)
 		(property "Capacitance (Farad)" "1µF"
-			(at 181.61 60.3249 90)
+			(at 165.1 59.0549 90)
 			(effects
 				(font
@@
 		)
 		(property "Tolerance (%)" "±20%"
-			(at 180.848 53.086 0)
+			(at 164.338 51.816 0)
 			(effects
 				(font
@@
 		)
 		(property "Voltage Rated (Volt)" "25V"
-			(at 182.626 59.69 0)
+			(at 166.116 58.42 0)
 			(effects
 				(font
@@
 	(symbol
 		(lib_id "Capacitors:885012207098")
-		(at 186.69 58.42 90)
+		(at 170.18 57.15 90)
 		(unit 1)
 		(exclude_from_sim no)
@@
 		(fields_autoplaced yes)
 		(property "Reference" "C102"
-			(at 190.5 57.7849 90)
+			(at 173.99 56.5149 90)
 			(effects
 				(font
@@
 		)
 		(property "Value" "885012207098"
-			(at 195.58 59.69 0)
+			(at 179.07 58.42 0)
 			(effects
 				(font
@@
 		)
 		(property "Footprint" "Capacitors:C0805"
-			(at 210.82 59.69 0)
+			(at 194.31 58.42 0)
 			(effects
 				(font
@@
 		)
 		(property "Datasheet" "D"
-			(at 213.36 59.69 0)
+			(at 196.85 58.42 0)
 			(effects
 				(font
@@
 		)
 		(property "Description" "CAP CER 0.1UF 100nF 50V X7R 0805"
-			(at 208.28 59.69 0)
+			(at 191.77 58.42 0)
 			(effects
 				(font
@@
 		)
 		(property "Supplier" "Digikey"
-			(at 198.12 59.69 0)
+			(at 181.61 58.42 0)
 			(effects
 				(font
@@
 		)
 		(property "Supplier Part Number" "732-8080-1-ND"
-			(at 200.66 59.69 0)
+			(at 184.15 58.42 0)
 			(effects
 				(font
@@
 		)
 		(property "Manufacturer" "Wurth Electronics Inc."
-			(at 203.2 59.69 0)
+			(at 186.69 58.42 0)
 			(effects
 				(font
@@
 		)
 		(property "Manufacturer Part Number" "885012207098"
-			(at 205.74 59.69 0)
+			(at 189.23 58.42 0)
 			(effects
 				(font
@@
 		)
 		(property "Capacitance (Farad)" "100nF"
-			(at 190.5 60.3249 90)
+			(at 173.99 59.0549 90)
 			(effects
 				(font
@@
 		)
 		(property "Tolerance (%)" "±10%"
-			(at 189.738 53.086 0)
+			(at 173.228 51.816 0)
 			(effects
 				(font
@@
 		)
 		(property "Voltage Rated (Volt)" "50V"
-			(at 191.516 59.69 0)
-			(effects
-				(font
+			(at 175.006 58.42 0)
+			(effects
+				(font
